File: prototype/stlink.kicad_sch (KiCad schematic)
At the start: 53 parts, among them J1 Conn_01x04, J2 USB_OTG, J3 SWD, Q1 BC817, SW1 SW_Push, U2 STM32F103CBUx, U6 LD3985M33R_SOT23, Y2 8MHz

Commit message: nrf5240
Parts:
- added TP1: SWDIO, symbol Connector:TestPoint
- added TP2: SWCLK, symbol Connector:TestPoint
- added TP3: GND, symbol Connector:TestPoint
- added TP4: 3V3_STLINK, symbol Connector:TestPoint
Connections:
- net 3V3_STLINK: now also TP4.1
- net GND: now also TP3.1
- net STL_T_JTCK: now also TP2.1
- net STL_T_JTMS: now also TP1.1
Changed lines of the file:
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@@
     (stroke (width 0) (type default))
   )
-  (wire (pts (xy 68.58 71.12) (xy 82.55 71.12))
+  (wire (pts (xy 68.58 71.12) (xy 88.9 71.12))
     (stroke (width 0) (type default))
   )
@@
     (stroke (width 0) (type default))
   )
+  (wire (pts (xy 88.9 68.58) (xy 86.36 68.58))
+    (stroke (width 0) (type default))
+  )
   (wire (pts (xy 149.86 104.14) (xy 143.51 104.14))
     (stroke (width 0) (type default))
@@
     (stroke (width 0) (type default))
   )
+  (wire (pts (xy 86.36 66.04) (xy 86.36 68.58))
+    (stroke (width 0) (type default))
+  )
   (wire (pts (xy 68.58 63.5) (xy 82.55 63.5))
     (stroke (width 0) (type default))
@@
     (stroke (width 0) (type default))
   )
-  (wire (pts (xy 68.58 73.66) (xy 82.55 73.66))
+  (wire (pts (xy 68.58 73.66) (xy 88.9 73.66))
     (stroke (width 0) (type default))
   )
@@
     (stroke (width 0) (type default))
   )
+  (wire (pts (xy 86.36 76.2) (xy 86.36 78.74))
+    (stroke (width 0) (type default))
+  )
   (wire (pts (xy 165.1 86.36) (xy 165.1 88.9))
     (stroke (width 0) (type default))
@@
     (stroke (width 0) (type default))
   )
+  (wire (pts (xy 88.9 76.2) (xy 86.36 76.2))
+    (stroke (width 0) (type default))
+  )
   (wire (pts (xy -114.3 139.7) (xy -114.3 142.24))
     (stroke (width 0) (type default))
@@
     (effects (font (size 1.27 1.27)) (justify right bottom))
   )
-  (text "SWCLK" (at 83.82 73.66 0)
-    (effects (font (size 1.27 1.27)) (justify left bottom))
-  )
   (text "?" (at -113.03 128.27 0)
     (effects (font (size 1.27 1.27)) (justify left bottom))
@@
     (effects (font (size 1.27 1.27)) (justify left bottom))
   )
-  (text "SWDIO" (at 83.82 71.12 0)
-    (effects (font (size 1.27 1.27)) (justify left bottom))
-  )
   (text "T_JTDO" (at 69.85 53.34 0)
     (effects (font (size 1.27 1.27)) (justify left bottom))
@@
     (effects (font (size 1.27 1.27)) (justify left bottom))
   )
+  (label "3V3_STLINK" (at 86.36 66.04 0) (fields_autoplaced)
+    (effects (font (size 1.27 1.27)) (justify left bottom))
+  )
   (label "STL_USB_D_N" (at 160.02 109.22 180) (fields_autoplaced)
     (effects (font (size 1.27 1.27)) (justify right bottom))
@@
   (label "STL_T_JTCK" (at 19.05 99.06 0) (fields_autoplaced)
     (effects (font (size 1.27 1.27)) (justify left bottom))
+  )
+  (symbol (lib_id "Connector:TestPoint") (at 88.9 71.12 270) (unit 1)
+    (in_bom yes) (on_board yes) (dnp no)
+    (property "Reference" "TP1" (at 88.9 69.85 90)
+      (effects (font (size 1.27 1.27)))
+    )
+    (property "Value" "SWDIO" (at 93.98 71.12 90)
+      (effects (font (size 1.27 1.27)) (justify left))
+    )
+    (property "Footprint" "" (at 88.9 76.2 0)
+      (effects (font (size 1.27 1.27)) hide)
+    )
+    (property "Datasheet" "~" (at 88.9 76.2 0)
+      (effects (font (size 1.27 1.27)) hide)
+    )
+    (pin "1")
+    (instances
+      (project "main"
+        (path "/71bbf5b6-a913-4747-956a-150714430eae/8c222416-b30d-49c6-bdd9-9c9a8764b515"
+          (reference "TP1") (unit 1)
+        )
+      )
+    )
   )
   (symbol (lib_id "Device:LED") (at 247.65 38.1 0) (unit 1)
@@
     )
   )
+  (symbol (lib_id "power:GND") (at 86.36 78.74 0) (unit 1)
+    (in_bom yes) (on_board yes) (dnp no)
+    (property "Reference" "#PWR043" (at 86.36 85.09 0)
+      (effects (font (size 1.27 1.27)) hide)
+    )
+    (property "Value" "GND" (at 86.36 82.55 0)
+      (effects (font (size 1.27 1.27)))
+    )
+    (property "Footprint" "" (at 86.36 78.74 0)
+      (effects (font (size 1.27 1.27)) hide)
+    )
+    (property "Datasheet" "" (at 86.36 78.74 0)
+      (effects (font (size 1.27 1.27)) hide)
+    )
+    (pin "1")
+    (instances
+      (project "main"
+        (path "/71bbf5b6-a913-4747-956a-150714430eae/8c222416-b30d-49c6-bdd9-9c9a8764b515"
+          (reference "#PWR043") (unit 1)
+        )
+      )
+    )
+  )
   (symbol (lib_id "Device:R") (at 234.95 38.1 90) (unit 1)
     (in_bom yes) (on_board yes) (dnp no)
@@
         (path "/71bbf5b6-a913-4747-956a-150714430eae/8c222416-b30d-49c6-bdd9-9c9a8764b515"
           (reference "R17") (unit 1)
+        )
+      )
+    )
+  )
+  (symbol (lib_id "Connector:TestPoint") (at 88.9 73.66 270) (unit 1)
+    (in_bom yes) (on_board yes) (dnp no)
+    (property "Reference" "TP2" (at 88.9 72.39 90)
+      (effects (font (size 1.27 1.27)))
+    )
+    (property "Value" "SWCLK" (at 93.98 73.66 90)
+      (effects (font (size 1.27 1.27)) (justify left))
+    )
+    (property "Footprint" "" (at 88.9 78.74 0)
+      (effects (font (size 1.27 1.27)) hide)
+    )
+    (property "Datasheet" "~" (at 88.9 78.74 0)
+      (effects (font (size 1.27 1.27)) hide)
+    )
+    (pin "1")
+    (instances
+      (project "main"
+        (path "/71bbf5b6-a913-4747-956a-150714430eae/8c222416-b30d-49c6-bdd9-9c9a8764b515"
+          (reference "TP2") (unit 1)
         )
       )
@@
         (path "/71bbf5b6-a913-4747-956a-150714430eae/8c222416-b30d-49c6-bdd9-9c9a8764b515"
           (reference "Y2") (unit 1)
+        )
+      )
+    )
+  )
+  (symbol (lib_id "Connector:TestPoint") (at 88.9 76.2 270) (unit 1)
+    (in_bom yes) (on_board yes) (dnp no)
+    (property "Reference" "TP3" (at 88.9 74.93 90)
+      (effects (font (size 1.27 1.27)))
+    )
+    (property "Value" "GND" (at 93.98 76.2 90)
+      (effects (font (size 1.27 1.27)) (justify left))
+    )
+    (property "Footprint" "" (at 88.9 81.28 0)
+      (effects (font (size 1.27 1.27)) hide)
+    )
+    (property "Datasheet" "~" (at 88.9 81.28 0)
+      (effects (font (size 1.27 1.27)) hide)
+    )
+    (pin "1")
+    (instances
+      (project "main"
+        (path "/71bbf5b6-a913-4747-956a-150714430eae/8c222416-b30d-49c6-bdd9-9c9a8764b515"
+          (reference "TP3") (unit 1)
         )
       )
@@
         )
       )
+    )
+  )
+  (symbol (lib_id "Connector:TestPoint") (at 88.9 68.58 270) (unit 1)
+    (in_bom yes) (on_board yes) (dnp no)
+    (property "Reference" "TP4" (at 88.9 67.31 90)
+      (effects (font (size 1.27 1.27)))
+    )
+    (property "Value" "3V3_STLINK" (at 93.98 68.58 90)
+      (effects (font (size 1.27 1.27)) (justify left))
+    )
+    (property "Footprint" "" (at 88.9 73.66 0)
+      (effects (font (size 1.27 1.27)) hide)
+    )
+    (property "Datasheet" "~" (at 88.9 73.66 0)
+      (effects (font (size 1.27 1.27)) hide)
+    )
+    (pin "1")
+    (instances
+      (project "main"
+        (path "/71bbf5b6-a913-4747-956a-150714430eae/8c222416-b30d-49c6-bdd9-9c9a8764b515"
+          (reference "TP4") (unit 1)
+        )
+      )
