File: prototype/usb_iso.kicad_sch (KiCad schematic)
At the start: 0 parts

Commit message: DAPLink, FT2232H
Parts:
- added D14: SK24A, Diode_SMD:D_SMA, symbol Device:D_Schottky
- added J7: TYPE-C-31-M-12, MAS_Package_std:USB_C_Receptacle_HRO_TYPE-C-31-M-12, symbol Connector:USB_C_Receptacle_USB2.0
- added R62 (x2): 22k, Resistor_SMD:R_0603_1608Metric, symbol Device:R
Connections:
- new net: D14.2 (A), J7.A4 (VBUS), J7.A9 (VBUS), J7.B4 (VBUS), J7.B9 (VBUS)
- new net +5V: D14.1 (K)
- new net CC1: J7.A5 (CC1), R62.1
- new net CC2: J7.B5 (CC2), R62.1
- new net GND: J7.A1 (GND), J7.A12 (GND), J7.B1 (GND), J7.B12 (GND), J7.S1 (SHIELD), R62.2, R62.2
- new net PC_USB_N: J7.A7 (D-), J7.B7 (D-)
- new net PC_USB_P: J7.A6 (D+), J7.B6 (D+)
- no-connect marks 0 -> 2
