File: prototype/rs485.kicad_sch (KiCad schematic)
At the start: 12 parts, among them J501 RS485, U501 TBU-CA065-200-WH, U502 TBU-CA065-200-WH, U503 SN65HVD75D

Commit message: tmp
Parts:
- removed C501: 0.1u, Capacitor_SMD:C_0603_1608Metric, symbol Device:C
- removed D501: CDSOT23-SM712, Package_TO_SOT_SMD:SOT-23, symbol Diode:SM712_SOT23
- removed J501: RS485, symbol Connector:Screw_Terminal_01x03
- removed JP1: 120 Ohm, Jumper:SolderJumper-2_P1.3mm_Open_RoundedPad1.0x1.5mm, symbol Jumper:SolderJumper_2_Open
- removed R501: 120, Resistor_SMD:R_0805_2012Metric, symbol Device:R
- removed R502, R503: 10, Resistor_SMD:R_0603_1608Metric, symbol Device:R
- removed RV501, RV502: VC120626D580DP, Resistor_SMD:R_1206_3216Metric, symbol Device:Varistor
- removed U501, U502: TBU-CA065-200-WH, chrns_nostd:TBU-CAxxx-xxx-WH, symbol chrns_ic_power:TBU
- removed U503: SN65HVD75D, Package_SO:SOIC-8_3.9x4.9mm_P1.27mm, symbol chrns_ic_connectivity:SN65HVD75D
- added C?: 0.1u, Capacitor_SMD:C_0603_1608Metric, symbol Device:C
- added D?: FYLS-0603BURC, LED_SMD:LED_0603_1608Metric, symbol Device:LED
- added D?: CDSOT23-SM712, Package_TO_SOT_SMD:SOT-23, symbol Diode:SM712_SOT23
- added D?: FYLS-0603BPGC, LED_SMD:LED_0603_1608Metric, symbol Device:LED
- added J?: ED350V-03P, chrns_nostd:ED350V-03P, symbol Connector:Screw_Terminal_01x03
- added JP?: TRM, Jumper:SolderJumper-2_P1.3mm_Open_RoundedPad1.0x1.5mm, symbol Jumper:SolderJumper_2_Open
- added R? (x2): 10, Resistor_SMD:R_0603_1608Metric, symbol Device:R
- added R? (x2): 560, Resistor_SMD:R_0603_1608Metric, symbol Device:R
- added R?: 120, Resistor_SMD:R_0805_2012Metric, symbol Device:R
- added RV? (x2): VC120626D580DP, Resistor_SMD:R_1206_3216Metric, symbol Device:Varistor
- added U23: SN65HVD75DRBR, Package_SON:Texas_S-PVSON-N8, symbol chrns_ic_connectivity:SN65HVD75D
- added U? (x2): TBU-CA065-200-WH, chrns_nostd:TBU-CAxxx-xxx-WH, symbol chrns_ic_power:TBU
Connections:
- net FT_DTR: now also U23.2 (~{RE}), U23.3 (DE)
- net FT_RXD: now also U23.1 (R)
- net FT_TXD: now also U23.4 (D)
- net GND: now also C?.2, U23.5 (GND)
- net RS485_A: now also R?.2, U23.6 (A)
- net RS485_B: now also R?.2, U23.7 (B)
- net RS485_IN_A: now also J?.1 (Pin_1), RV?.2, U?.1
- net RS485_IN_B: now also J?.3 (Pin_3), RV?.1, U?.1
- net RS485_IN_G: now also D?.3 (common), J?.2 (Pin_2), RV?.1, RV?.2
- new net: D?.1 (A1), R?.1, R?.1, U?.3
- new net: D?.2 (A2), JP?.1 (A), R?.1, U?.3
- new net: JP?.2 (B), R?.2
- new net: D?.2 (A), R?.1 (x2)
- new net 3V3D_HUB: C?.1, R?.2, R?.2, U23.8 (VCC)
- new net RS_LED_R: D?.1 (K)
- new net RS_LED_T: D?.1 (K)
