File: prototype/ble.kicad_sch (KiCad schematic)
At the start: 2 parts, among them U3 nRF52840, U4 STM32WB55CCUx

Commit message: nrf5240
Parts:
- removed U4: STM32WB55CCUx, Package_DFN_QFN:QFN-48-1EP_7x7mm_P0.5mm_EP5.6x5.6mm, symbol MCU_ST_STM32WB:STM32WB55CCUx
- added AE1: Antenna, symbol Device:Antenna
- added C55: 0.8p, symbol Device:C
- added C56: 0.5p, symbol Device:C
- added C57, C? (x3): N.C., symbol Device:C
- added C6 (x2), C7 (x2): 12p, symbol Device:C
- added C77, C78: C, symbol Device:C
- added C? (x5): 0.1u, symbol Device:C
- added C? (x4): 4.7u, symbol Device:C
- added C?: 47n, symbol Device:C
- added C? (x2): 1u, symbol Device:C
- added D?: FYLS-3528RGBC, LED_SMD:LED_Kingbright_AAA3528ESGCT, symbol Device:LED_RABG
- added J7: NRF_SWD, symbol Connector_Generic:Conn_02x05_Odd_Even
- added J8: Conn_01x02, symbol Connector_Generic:Conn_01x02
- added L3: 4.7u, symbol Device:L
- added L4, L6: 10u, symbol Device:L
- added L5: 15n, symbol Device:L
- added R61: 100k, symbol Device:R
- added R62, R63: 0, symbol Device:R
- added R? (x3): 330, Resistor_SMD:R_0603_1608Metric, symbol Device:R
- added Y2: 32 MHz, symbol Device:Crystal_GND24
- added Y2: 32.768 kHz, symbol Device:Crystal_GND24
Connections:
- net NRF_DEC2: now reaches U3.A18 (DEC2)
- net NRF_DEC2: now also C?.1
- net VDD_NRF: now reaches U3.A22 (VDD), U3.AD14 (VDD), U3.AD23 (VDD), U3.B1 (VDD), U3.W1 (VDD)
- net VDD_NRF: now also C?.1, C?.1, C?.1, C?.1, C?.1, L6.1
- net NRF_XC2: now reaches U3.A23 (XC2)
- net NRF_XC2: now also C7.1, Y2.1
- net NRF_SWCLK: now reaches U3.AA24 (SWDCLK)
- net NRF_DCCH: now reaches U3.AB2 (DCCH)
- net NRF_DCCH: now also L6.2
- net NRF_NRST: now reaches U3.AC13 (P0.18/~{RESET})
- net NRF_SWDIO: now reaches U3.AC24 (SWDIO)
- net DECUSB: now reaches U3.AC5 (DECUSB)
- net DECUSB: now also C?.1
- net VBUS_NRF: now reaches U3.AD2 (VBUS)
- net VBUS_NRF: now also C?.1
- net NRF_SWO: now reaches U3.AD22 (TRACEDATA0/P1.00)
- net NRF_USB_D_N: now reaches U3.AD4 (D-)
- net NRF_USB_D_P: now reaches U3.AD6 (D+)
- net NRF_XC1: now reaches U3.B24 (XC1)
- net NRF_XC1: now also C6.1, Y2.3
- net NRF_DCC: now reaches U3.B3 (DCC)
- net NRF_DCC: now also L4.2
- net NRF_DEC4/6: now reaches U3.B5 (DEC4)
- net NRF_DEC4/6: now also U3.E24 (DEC6), C?.1, C?.1, C?.1, L5.1
- net GND: now reaches U3.B7 (VSS), U3.EP (VSS)
- net GND: now also U3.F23 (VSS_PA), C55.2, C56.2, C57.2, C6.2, C6.2, C7.2, C7.2, C77.2, C78.2, C?.2, C?.2, C?.2, C?.2, C?.2, C?.2, C?.2, C?.2, C?.2, C?.2, J7.5 (Pin_5), Y2.2, Y2.2, Y2.4, Y2.4
- net NRF_DEC1: now reaches U3.C1 (DEC1)
- net NRF_DEC1: now also C?.1
- net NRF_XL1: now reaches U3.D2 (XL1/P0.00)
- net NRF_XL1: now also C6.1, Y2.3
- net NRF_DEC3: now reaches U3.D23 (DEC3)
- net NRF_DEC3: now also C?.1
- net NRF_XL2: now reaches U3.F2 (XL2/P0.01)
- net NRF_XL2: now also C7.1, Y2.1
- net NRF_SDA: now reaches U3.G1 (P0.26)
- net NRF_SCL: now reaches U3.H2 (P0.27)
- net NRF_ANT: now reaches U3.H23 (ANT)
- net NRF_ANT: now also C55.1, L3.1
- net NRF_NFC2: now reaches U3.J24 (NFC2/P0.10)
- net NRF_NFC2: now also R63.1
- net NRF_NFC1: now reaches U3.L24 (NFC1/P0.09)
- net NRF_NFC1: now also R62.1
- net NRF_T_CLK: now reaches U3.M2 (TRACECLK/P0.07)
- net NRF_DEC5: now reaches U3.N24 (DEC5)
- net NRF_DEC5: now also C?.1
- net NRF_T_DAT3: now reaches U3.R1 (TRACEDATA3/P1.09)
- net NRF_T_DAT2: now reaches U3.T2 (TRACEDATA2/P0.11)
- net NRF_T_DAT1: now reaches U3.U1 (TRACEDATA1/P0.12)
- net VDD_HV: now reaches U3.Y2 (VDDH)
- net VDD_HV: now also C?.1
- new net: AE1.1 (A), C56.1, C57.1, L3.2
- new net: C?.2, C?.2, C?.2, C?.2, C?.2
- new net: D?.4 (GK), R?.2
- new net: L4.1, L5.2
- new net: D?.1 (RK), R?.2
- new net: D?.3 (BK), R?.2
- new net +3.3V: D?.2 (A)
- new net IMCU_RESET: J7.2 (Pin_2), R61.2
- new net IMCU_SWDCLK: J7.7 (Pin_7)
- new net IMCU_SWDIO: J7.3 (Pin_3)
- new net LED_B_L: R?.1
- new net LED_G_L: R?.1
- new net LED_R_L: R?.1
- new net NFC_ANT1: C78.1, J8.1 (Pin_1), R62.2
- new net NFC_ANT2: C77.1, J8.2 (Pin_2), R63.2
- new net VBUS: J7.9 (Pin_9)
- new net VDD_IMCU: J7.1 (Pin_1), R61.1
- no-connect marks 0 -> 4
Other:
- note added: "A22"
- note added: "AD14"
- note added: "AD23"
- note added: "B1"
- note added: "Interfaces: I2C, SPI/QSPI, 1-Wire, UART Timers: PWM, Servo tester, Freq.Meter/Duty Cycle meter, PWM + Dead time Analog: ADC, Comparator ... DAC (external IC)"
- note added: "trace to stlink via jupmers"
- moved on the sheet: U3

Commit message: DAPLink, FT2232H
Parts:
- added J10: I2C, symbol Connector_Generic:Conn_01x04
- added J11: 1-Wire, symbol Connector_Generic:Conn_01x03
- added J12: Conn_01x05, symbol Connector_Generic:Conn_01x05
- added J14: Conn_01x08, symbol Connector_Generic:Conn_01x08
- added J19, J2: Micro_SD_Card_Det1, symbol Connector:Micro_SD_Card_Det1
- added R11, R12, R13 (x3): 47k, symbol Device:R
- added R57, R58, R59, R68: 4.7k, symbol Device:R
- added R60, R64, R65, R66, R67: 22, symbol Device:R
- added RN1: R_Pack04, symbol Device:R_Pack04
- added SW6: Mode, symbol Switch:SW_DIP_x04
- added Y4: NX3215SA-32.768, MAS_Package_std:Crystal_SMD_3215-2Pin_3.2x1.5mm, symbol Device:Crystal
- D?: chipdip 8001774353 -> (none); elitan 9838555 -> (none); promelec 337147 -> (none)
- J8: value Conn_01x02 -> NFC
- R? (x3): Accuracy ±5% -> (none); Part number RC0603JR-07220RL -> (none); chipdip 8008270850 -> (none); elitan 618023 -> (none); lcsc C114683 -> (none); promelec 19859 -> (none)
Connections:
- net GND: now also C?.2, C?.2, C?.2, C?.2, C?.2, J10.4 (Pin_4), J11.3 (Pin_3), J14.8 (Pin_8), J2.10 (SHIELD), J2.6 (VSS), R68.2
- net NRF_SCL: now also J10.3 (Pin_3), R58.2
- net NRF_SDA: now also J10.2 (Pin_2), R57.2
- net NRF_SWO: now also J12.2 (Pin_2)
- net NRF_T_CLK: now also J12.1 (Pin_1)
- net NRF_T_DAT1: now also J12.3 (Pin_3)
- net NRF_T_DAT3: now also J12.4 (Pin_4), J12.5 (Pin_5)
- net VDD_NRF: now also J10.1 (Pin_1), J11.1 (Pin_1), J14.1 (Pin_1), R57.1, R58.1, R59.1
- new net: R68.1, SW6.5, SW6.6, SW6.7, SW6.8
- new net NFC_QSPI_CLK: J14.2 (Pin_2)
- new net NFC_QSPI_CS: J14.7 (Pin_7)
- new net NFC_QSPI_IO0/SO: J14.3 (Pin_3)
- new net NFC_QSPI_IO1/SI: J14.4 (Pin_4)
- new net NFC_QSPI_IO2/WP: J14.5 (Pin_5)
- new net NFC_QSPI_IO3/HOLD: J14.6 (Pin_6)
- new net NRF_MODE0: SW6.1
- new net NRF_MODE1: SW6.2
- new net NRF_MODE2: SW6.3
- new net NRF_MODE3: SW6.4
- new net ONE_WIRE: J11.2 (Pin_2), R59.2
- new net VCC_3V3: J2.4 (VDD), R11.2, R12.2, R13.2, R13.2, R13.2
- new net uSD_CS: J2.2 (DAT3/CD), R11.1
- new net uSD_DET: J2.9 (DET), R13.1
- new net uSD_DI: J2.3 (CMD), R12.1
- new net uSD_DO: J2.7 (DAT0), R13.1
- new net uSD_SCK: J2.5 (CLK), R13.1
- no-connect marks 4 -> 6
Other:
- note added: "??"
- note added: "ESD"
- note added: "Interfaces: I2C, SPI/QSPI, 1-Wire, UART Timers: PWM, Servo tester, Freq.Meter/Duty Cycle meter, PWM + Dead time Analog: ADC, Comparator ... DAC (external IC) Other: EEPROM/SPI programmer"
- note added: "SD Card nRF52840 P1.12 - D3/CS P1.13 - DI/MOSI P1.15 - CLK P1.14 - D0/MISO"
- note added: "https://infocenter.nordicsemi.com/index.jsp?topic=%2Fcom.nordic.infocenter.sdk5.v13.0.0%2Fapp_sdcard_example.html"
- note removed: "Interfaces: I2C, SPI/QSPI, 1-Wire, UART Timers: PWM, Servo tester, Freq.Meter/Duty Cycle meter, PWM + Dead time Analog: ADC, Comparator ... DAC (external IC)"
- moved on the sheet: J7, R61

Commit message: tmp
Parts:
- removed J19: Micro_SD_Card_Det1, symbol Connector:Micro_SD_Card_Det1
Changed lines of the file:
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@@
   )
   (text "https://infocenter.nordicsemi.com/index.jsp?topic=%2Fcom.nordic.infocenter.sdk5.v13.0.0%2Fapp_sdcard_example.html"
-    (at 317.5 223.52 0)
+    (at 135.89 255.27 0)
     (effects (font (size 1.27 1.27)) (justify left bottom))
   )
@@
   )
   (text "SD Card nRF52840\nP1.12 - D3/CS\nP1.13 - DI/MOSI\nP1.15 - CLK\nP1.14 - D0/MISO"
-    (at 317.5 234.95 0)
+    (at 135.89 266.7 0)
     (effects (font (size 1.27 1.27)) (justify left bottom))
   )
@@
   (hierarchical_label "TRG_TXD" (shape output) (at -5.08 -2.54 180) (fields_autoplaced)
     (effects (font (size 1.27 1.27)) (justify right))
+  )
+  (hierarchical_label "BB_ADJ" (shape input) (at 12.7 -2.54 180) (fields_autoplaced)
+    (effects (font (size 1.27 1.27)) (justify right))
+  )
+  (hierarchical_label "PWR_STAT" (shape input) (at 12.7 -10.16 180) (fields_autoplaced)
+    (effects (font (size 1.27 1.27)) (justify right))
+  )
+  (hierarchical_label "NRF_PD_INT" (shape input) (at 116.84 110.49 0) (fields_autoplaced)
+    (effects (font (size 1.27 1.27)) (justify left))
   )
   (hierarchical_label "NRF_USB_D_N" (shape bidirectional) (at 99.06 165.1 0) (fields_autoplaced)
@@
     (effects (font (size 1.27 1.27)) (justify right))
   )
+  (hierarchical_label "NRF_PD_INT" (shape input) (at 12.7 -12.7 180) (fields_autoplaced)
+    (effects (font (size 1.27 1.27)) (justify right))
+  )
   (hierarchical_label "NRF_SCL" (shape bidirectional) (at 116.84 106.68 0) (fields_autoplaced)
     (effects (font (size 1.27 1.27)) (justify left))
   )
+  (hierarchical_label "LDO_ADJ" (shape input) (at 12.7 0 180) (fields_autoplaced)
+    (effects (font (size 1.27 1.27)) (justify right))
+  )
   (hierarchical_label "TRG_RXD" (shape input) (at -5.08 0 180) (fields_autoplaced)
+    (effects (font (size 1.27 1.27)) (justify right))
+  )
+  (hierarchical_label "PWR_EN" (shape input) (at 12.7 -7.62 180) (fields_autoplaced)
     (effects (font (size 1.27 1.27)) (justify right))
   )
   (hierarchical_label "NRF_SDA" (shape bidirectional) (at 116.84 104.14 0) (fields_autoplaced)
     (effects (font (size 1.27 1.27)) (justify left))
+  )
+  (hierarchical_label "EXT_PWR_CTRL" (shape input) (at 12.7 -5.08 180) (fields_autoplaced)
+    (effects (font (size 1.27 1.27)) (justify right))
   )
   (hierarchical_label "NRF_USB_D_P" (shape bidirectional) (at 99.06 167.64 0) (fields_autoplaced)
@@
         )
       )
-    )
-  )
-  (symbol (lib_id "Connector:Micro_SD_Card_Det1") (at 387.35 276.86 0) (unit 1)
-    (in_bom yes) (on_board yes) (dnp no)
-    (property "Reference" "J19" (at 370.84 259.08 0)
-      (effects (font (size 1.27 1.27)))
-    )
-    (property "Value" "Micro_SD_Card_Det1" (at 393.7 259.08 0)
-      (effects (font (size 1.27 1.27)))
-    )
-    (property "Footprint" "" (at 439.42 259.08 0)
-      (effects (font (size 1.27 1.27)) hide)
-    )
-    (property "Datasheet" "https://datasheet.lcsc.com/lcsc/2110151630_XKB-Connectivity-XKTF-015-N_C381082.pdf" (at 387.35 274.32 0)
-      (effects (font (size 1.27 1.27)) hide)
-    )
-    (pin "1")
-    (pin "10")
-    (pin "2")
-    (pin "3")
-    (pin "4")
-    (pin "5")
-    (pin "6")
-    (pin "7")
-    (pin "8")
-    (pin "9")
-    (instances
-      (project "main"
-        (path "/71bbf5b6-a913-4747-956a-150714430eae/435e72e9-c3db-4675-9207-615c69453003"
-          (reference "J19") (unit 1)
-        )
-      )

Commit message: tmp
Parts:
- added AE2: 2.4 GHz (PCB), RF_Antenna:Texas_SWRA117D_2.4GHz_Left, symbol Device:Antenna
- C55, C56, C57, C6, C7, C77, C78, C? (x15): footprint (none) -> Capacitor_SMD:C_0402_1005Metric
- R11, R12, R13, R57, R58, R59, R60, R61, R62, R63, R64, R65, R66, R67, R68: footprint (none) -> Resistor_SMD:R_0402_1005Metric
Other:
- note added: "ESP32-S3 ESP8265"
