File: prototype/bridge.kicad_sch (KiCad schematic)
At the start: 0 parts

Commit message: DAPLink, FT2232H
Parts:
- added C100, C102, C103, C92, C93, C94, C95, C96, C97, C98: 0.1u, symbol Device:C
- added C101, C91, C99: 4.7u, symbol Device:C
- added C54, C90: 12p, symbol Device:C
- added D16: RED, symbol Device:LED
- added D17: GREEN, symbol Device:LED
- added J24: FT2232H, symbol Connector_Generic:Conn_02x10_Counter_Clockwise
- added L7, L8: L, symbol Device:L
- added R72: 2.2k, symbol Device:R
- added R73, R74, R75, R89, R90: 10k, symbol Device:R
- added R91, R92: 1k, symbol Device:R
- added U14: 93LC56B, Package_TO_SOT_SMD:SOT-23-6, symbol Memory_EEPROM:93LCxxB
- added U15, U16: TXS0108ERGYR, Package_SO:TSSOP-20_4.4x6.5mm_P0.65mm, symbol Logic_LevelTranslator:TXS0108EPW
- added U8: FT2232HQ, Package_DFN_QFN:QFN-64-1EP_9x9mm_P0.5mm_EP4.35x4.35mm, symbol Interface_USB:FT2232HQ
- added Y9: 12MHz, symbol Device:Crystal_GND24
Connections:
- new net: D17.1 (K), R92.2
- new net: R72.1, U14.4 (DO)
- new net: R89.2, U8.14 (~{RESET})
- new net: R90.2, U8.6 (REF)
- new net: D16.1 (K), R91.2
- new net 1V8_FT: C91.1, C92.1, C93.1, C94.1, C95.1, U8.12 (VCORE), U8.37 (VCORE), U8.49 (VREGOUT), U8.64 (VCORE)
- new net 3V3_FT: C103.1, C96.1, C97.1, C98.1, D16.2 (A), D17.2 (A), L7.2, L8.1, R73.1, R74.1, R75.1, R89.1, U14.8 (VCC), U15.10 (OE), U15.2 (VCCA), U16.10 (OE), U16.2 (VCCA), U8.20 (VCCIO), U8.31 (VCCIO), U8.42 (VCCIO), U8.50 (VREGIN), U8.56 (VCCIO)
- new net CN_AD4: J24.20 (Pin_20), U15.15 (B5)
- new net CN_AD5: J24.19 (Pin_19), U15.14 (B6)
- new net CN_AD6: J24.18 (Pin_18), U15.13 (B7)
- new net CN_AD7: J24.17 (Pin_17), U15.12 (B8)
- new net CN_BD5: J24.15 (Pin_15), U16.14 (B6)
- new net CN_BD6: J24.14 (Pin_14), U16.13 (B7)
- new net CN_BD7: J24.13 (Pin_13), U16.12 (B8)
- new net CN_CTS: J24.8 (Pin_8), U16.16 (B4)
- new net CN_DTR: J24.16 (Pin_16), U16.15 (B5)
- new net CN_RTS: J24.7 (Pin_7), U16.17 (B3)
- new net CN_RXD: J24.6 (Pin_6), U16.18 (B2)
- new net CN_TCK: J24.1 (Pin_1), U15.20 (B1)
- new net CN_TDI: J24.2 (Pin_2), U15.18 (B2)
- new net CN_TDO: J24.3 (Pin_3), U15.17 (B3)
- new net CN_TMS: J24.4 (Pin_4), U15.16 (B4)
- new net CN_TXD: J24.5 (Pin_5), U16.20 (B1)
- new net FT_AD4: U15.6 (A5), U8.21 (ADBUS4)
- new net FT_AD5: U15.7 (A6), U8.22 (ADBUS5)
- new net FT_AD6: U15.8 (A7), U8.23 (ADBUS6)
- new net FT_AD7: U15.9 (A8), U8.24 (ADBUS7)
- new net FT_BD5: U16.7 (A6), U8.44 (BDBUS5)
- new net FT_BD6: U16.8 (A7), U8.45 (BDBUS6)
- new net FT_BD7: U16.9 (A8), U8.46 (BDBUS7)
- new net FT_CTS: U16.5 (A4), U8.41 (BDBUS3)
- new net FT_DTR: U16.6 (A5), U8.43 (BDBUS4)
- new net FT_EECLK: R74.2, U14.2 (SCLK), U8.62 (EECLK)
- new net FT_EECS: R73.2, U14.1 (CS), U8.63 (EECS)
- new net FT_EEDATA: R72.2, R75.2, U14.3 (DI), U8.61 (EEDATA)
- new net FT_OSC_I: C90.1, U8.2 (OSCI), Y9.3
- new net FT_OSC_O: C54.1, U8.3 (OSCO), Y9.1
- new net FT_RTS: U16.4 (A3), U8.40 (BDBUS2)
- new net FT_RXD: U16.3 (A2), U8.39 (BDBUS1)
- new net FT_RX_LED: R91.1, U8.54 (BCBUS3)
- new net FT_TCK: U15.1 (A1), U8.16 (ADBUS0)
- new net FT_TDI: U15.3 (A2), U8.17 (ADBUS1)
- new net FT_TDO: U15.4 (A3), U8.18 (ADBUS2)
- new net FT_TMS: U15.5 (A4), U8.19 (ADBUS3)
- new net FT_TXD: U16.1 (A1), U8.38 (BDBUS0)
- new net FT_TX_LED: R92.1, U8.55 (BCBUS4)
- new net FT_USB_D_N: U8.7 (DM)
- new net FT_USB_D_P: U8.8 (DP)
- new net GND: C100.2, C101.1, C102.1, C103.2, C54.2, C90.2, C91.2, C92.2, C93.2, C94.2, C95.2, C96.2, C97.2, C98.2, C99.2, J24.10 (Pin_10), J24.11 (Pin_11), J24.12 (Pin_12), J24.9 (Pin_9), R90.1, U14.5 (GND), U15.11 (GND), U16.11 (GND), U8.1 (GND), U8.10 (AGND), U8.11 (GND), U8.13 (TEST), U8.15 (GND), U8.25 (GND), U8.35 (GND), U8.47 (GND), U8.5 (GND), U8.51 (GND), U8.65 (GND), Y9.2, Y9.4
- new net VPHY_FT: C101.2, C102.2, L7.1, U8.4 (VPHY)
- new net VPLL_FT: C100.1, C99.1, L8.2, U8.9 (VPLL)
- no-connect marks 0 -> 16
Other:
- note added: "1.8V, 3.3V, 5V"
- note added: "C193662"
- note added: "C27882"
- note added: "FT2232HL"
- note added: "FT2232HQ"
- note added: "JTAG: - D0 == TCK - D1 == TDI - D2 == TDO - D3 == TMS"
- note added: "SPI: - D0 == SCK - D1 == MOSI - D2 == MISO - D3 == CS"
- note added: "TXS0108ERGYR"
- note added: "UART: - D0 == Tx - D1 == Rx"
- note added: "flashrom -p ft2232_spi:type=232H -r path/to/output/file.dat"

Commit message: tmp
Parts:
- C100, C101, C102, C103, C54, C90, C91, C92, C93, C94, C95, C96, C97, C98, C99: footprint (none) -> Capacitor_SMD:C_0402_1005Metric
- R72, R73, R74, R75, R89, R90, R91, R92: footprint (none) -> Resistor_SMD:R_0402_1005Metric
Changed lines of the file:
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@@
       (effects (font (size 1.27 1.27)) (justify left))
     )
-    (property "Footprint" "" (at 77.1652 181.61 0)
+    (property "Footprint" "Capacitor_SMD:C_0402_1005Metric" (at 77.1652 181.61 0)
       (effects (font (size 1.27 1.27)) hide)
     )
@@
       (effects (font (size 1.27 1.27)) (justify left))
     )
-    (property "Footprint" "" (at 204.1652 149.86 0)
+    (property "Footprint" "Capacitor_SMD:C_0402_1005Metric" (at 204.1652 149.86 0)
       (effects (font (size 1.27 1.27)) hide)
     )
@@
       (effects (font (size 1.27 1.27)))
     )
-    (property "Footprint" "" (at 57.15 184.658 90)
+    (property "Footprint" "Resistor_SMD:R_0402_1005Metric" (at 57.15 184.658 90)
       (effects (font (size 1.27 1.27)) hide)
     )
@@
       (effects (font (size 1.27 1.27)) (justify left))
     )
-    (property "Footprint" "" (at 166.0652 149.86 0)
+    (property "Footprint" "Capacitor_SMD:C_0402_1005Metric" (at 166.0652 149.86 0)
       (effects (font (size 1.27 1.27)) hide)
     )
@@
       (effects (font (size 1.27 1.27)) (justify left))
     )
-    (property "Footprint" "" (at 115.2652 187.96 0)
+    (property "Footprint" "Capacitor_SMD:C_0402_1005Metric" (at 115.2652 187.96 0)
       (effects (font (size 1.27 1.27)) hide)
     )
@@
       (effects (font (size 1.27 1.27)) (justify right))
     )
-    (property "Footprint" "" (at 240.3348 142.24 0)
+    (property "Footprint" "Capacitor_SMD:C_0402_1005Metric" (at 240.3348 142.24 0)
       (effects (font (size 1.27 1.27)) hide)
     )
@@
       (effects (font (size 1.27 1.27)) (justify right))
     )
-    (property "Footprint" "" (at 227.6348 142.24 0)
+    (property "Footprint" "Capacitor_SMD:C_0402_1005Metric" (at 227.6348 142.24 0)
       (effects (font (size 1.27 1.27)) hide)
     )
@@
       (effects (font (size 1.27 1.27)) (justify left))
     )
-    (property "Footprint" "" (at 267.6652 149.86 0)
+    (property "Footprint" "Capacitor_SMD:C_0402_1005Metric" (at 267.6652 149.86 0)
       (effects (font (size 1.27 1.27)) hide)
     )
@@
       (effects (font (size 1.27 1.27)) (justify left))
     )
-    (property "Footprint" "" (at 55.372 170.18 90)
+    (property "Footprint" "Resistor_SMD:R_0402_1005Metric" (at 55.372 170.18 90)
       (effects (font (size 1.27 1.27)) hide)
     )
@@
       (effects (font (size 1.27 1.27)) (justify left))
     )
-    (property "Footprint" "" (at 140.6652 149.86 0)
+    (property "Footprint" "Capacitor_SMD:C_0402_1005Metric" (at 140.6652 149.86 0)
       (effects (font (size 1.27 1.27)) hide)
     )
@@
       (effects (font (size 1.27 1.27)))
     )
-    (property "Footprint" "" (at 146.05 192.278 90)
+    (property "Footprint" "Resistor_SMD:R_0402_1005Metric" (at 146.05 192.278 90)
       (effects (font (size 1.27 1.27)) hide)
     )
@@
       (effects (font (size 1.27 1.27)) (justify left))
     )
-    (property "Footprint" "" (at 216.8652 149.86 0)
+    (property "Footprint" "Capacitor_SMD:C_0402_1005Metric" (at 216.8652 149.86 0)
       (effects (font (size 1.27 1.27)) hide)
     )
@@
       (effects (font (size 1.27 1.27)) (justify left))
     )
-    (property "Footprint" "" (at 153.3652 149.86 0)
+    (property "Footprint" "Capacitor_SMD:C_0402_1005Metric" (at 153.3652 149.86 0)
       (effects (font (size 1.27 1.27)) hide)
     )
@@
       (effects (font (size 1.27 1.27)))
     )
-    (property "Footprint" "" (at 146.05 179.578 90)
+    (property "Footprint" "Resistor_SMD:R_0402_1005Metric" (at 146.05 179.578 90)
       (effects (font (size 1.27 1.27)) hide)
     )
@@
       (effects (font (size 1.27 1.27)) (justify left))
     )
-    (property "Footprint" "" (at 49.022 170.18 90)
+    (property "Footprint" "Resistor_SMD:R_0402_1005Metric" (at 49.022 170.18 90)
       (effects (font (size 1.27 1.27)) hide)
     )
@@
       (effects (font (size 1.27 1.27)) (justify left))
     )
-    (property "Footprint" "" (at 191.4652 149.86 0)
+    (property "Footprint" "Capacitor_SMD:C_0402_1005Metric" (at 191.4652 149.86 0)
       (effects (font (size 1.27 1.27)) hide)
     )
@@
       (effects (font (size 1.27 1.27)) (justify left))
     )
-    (property "Footprint" "" (at 102.5652 187.96 0)
+    (property "Footprint" "Capacitor_SMD:C_0402_1005Metric" (at 102.5652 187.96 0)
       (effects (font (size 1.27 1.27)) hide)
     )
@@
       (effects (font (size 1.27 1.27)) (justify left))
     )
-    (property "Footprint" "" (at 280.3652 149.86 0)
+    (property "Footprint" "Capacitor_SMD:C_0402_1005Metric" (at 280.3652 149.86 0)
       (effects (font (size 1.27 1.27)) hide)
     )
@@
       (effects (font (size 1.27 1.27)) (justify left))
     )
-    (property "Footprint" "" (at 178.7652 149.86 0)
+    (property "Footprint" "Capacitor_SMD:C_0402_1005Metric" (at 178.7652 149.86 0)
       (effects (font (size 1.27 1.27)) hide)
     )
@@
       (effects (font (size 1.27 1.27)) (justify left))
     )
-    (property "Footprint" "" (at 23.622 170.18 90)
+    (property "Footprint" "Resistor_SMD:R_0402_1005Metric" (at 23.622 170.18 90)
       (effects (font (size 1.27 1.27)) hide)
     )
@@
       (effects (font (size 1.27 1.27)) (justify left))
     )
-    (property "Footprint" "" (at 127.9652 149.86 0)
+    (property "Footprint" "Capacitor_SMD:C_0402_1005Metric" (at 127.9652 149.86 0)
       (effects (font (size 1.27 1.27)) hide)
     )
@@
       (effects (font (size 1.27 1.27)))
     )
-    (property "Footprint" "" (at 38.1 72.898 90)
+    (property "Footprint" "Resistor_SMD:R_0402_1005Metric" (at 38.1 72.898 90)
       (effects (font (size 1.27 1.27)) hide)
     )
@@
       (effects (font (size 1.27 1.27)))
     )
-    (property "Footprint" "" (at 38.1 77.978 90)
-      (effects (font (size 1.27 1.27)) hide)
-    )
+    (property "Footprint" "Resistor_SMD:R_0402_1005Metric" (at 38.1 77.978 90)
+      (effects (font (size 1.27 1.27)) hide)
+    )
