File: prototype/daplink.kicad_sch (KiCad schematic)
At the start: 57 parts, among them J1 Conn_01x04, J2 USB_OTG, J3 SWD, Q1 BC817, SW1 SW_Push, U2 STM32F103CBUx, U6 LD3985M33R_SOT23, Y2 8MHz

Commit message: DAPLink, FT2232H
Parts:
- added J21: BMP, symbol Connector_Generic:Conn_02x05_Odd_Even
- added JP2: SWDIO, Jumper:SolderJumper-2_P1.3mm_Open_TrianglePad1.0x1.5mm, symbol Jumper:SolderJumper_2_Open
- added JP3: SWCLK, Jumper:SolderJumper-2_P1.3mm_Open_TrianglePad1.0x1.5mm, symbol Jumper:SolderJumper_2_Open
- added R56, R84, R85: 22, symbol Device:R
- added TP5: NRST, symbol Connector:TestPoint
- added U15: TXS0108ERGYR, Package_SO:TSSOP-20_4.4x6.5mm_P0.65mm, symbol Logic_LevelTranslator:TXS0108EPW
- TP1, TP2, TP3: now left out of the parts list
- TP4: value 3V3_STLINK -> 3V3_DAP; now left out of the parts list
- U6: value LD3985M33R_SOT23 -> LD3985M33R; lcsc (none) -> C46243
Connections:
- net 3V3_STLINK is gone; now on net 3V3_DAP: C12.1, C13.1, C2.1, C3.1, C4.1, C5.1, D4.2 (A), Q1.3 (C), R4.1, TP4.1, U2.1 (VBAT), U2.24 (VDD), U2.36 (VDD), U2.48 (VDD), U2.9 (VDDA), U6.5 (VOUT)
- net GND: now also J21.1 (Pin_1), U15.11 (GND)
- net TRG_CLK: now reaches J3.2 (Pin_2), R22.1
- net TRG_CLK: now also J21.10 (Pin_10), U15.3 (A2)
- net TRG_SWO: now reaches J3.6 (Pin_6), R19.1
- net TRG_SWO: now also J21.7 (Pin_7), U15.5 (A4)
- net TRG_DIO: now reaches J3.4 (Pin_4), R21.1
- net TRG_DIO: now also J21.9 (Pin_9), U15.4 (A3)
- net 3V3_DAP: now reaches J1.1 (Pin_1)
- net +3.3V: no longer names the net of R5.1
- net +5V: no longer names the net of R8.1
- net MCO renamed TRG_MCO
- net STL_AIN_1 renamed DAP_TRG_AIN
- net STL_BOOT0 renamed DAP_BOOT0
- net STL_LED renamed DAP_PRG_LED
- net STL_MCO renamed DAP_TRG_MCO
- net STL_NRST renamed DAP_NRST
- net DAP_NRST: now also TP5.1
- net STL_OSC_I renamed DAP_OSC_I
- net STL_OSC_O renamed DAP_OSC_O
- net STL_PC13 renamed DAP_PC13
- net STL_PC14 renamed DAP_PC14
- net STL_PWR_EXT renamed DAP_PWR_EXT
- net STL_RXD renamed DAP_TRG_RXD
- net DAP_TRG_RXD: now also R84.1; no longer J1.3 (Pin_3)
- net STL_TXD renamed DAP_TRG_TXD
- net DAP_TRG_TXD: now also R56.1, R85.2; no longer J1.2 (Pin_2)
- net STL_T_JTCK renamed DAP_TRG_CLK
- net DAP_TRG_CLK: now also JP3.2 (B); no longer TP2.1, U2.37 (PA14)
- net STL_T_JTMS renamed DAP_TRG_DIO
- net DAP_TRG_DIO: now also JP2.2 (B); no longer TP1.1, U2.34 (PA13)
- net STL_T_NRST renamed DAP_TRG_NRST
- net STL_T_SWDIO_IN renamed DAP_TRG_DIO_IN
- net STL_T_SWO renamed DAP_TRG_SWO
- net STL_USB_D_N renamed DAP_USB_D_N
- net STL_USB_D_P renamed DAP_USB_D_P
- net STL_USB_REN renamed DAP_USB_REN
- net TAR_NRST renamed TRG_RST
- net TRG_RST: now also U15.1 (A1)
- new net 3V3_FT: U15.2 (VCCA)
- new net 3V3_TRG: J21.3 (Pin_3)
- new net DAP_SWCLK: JP3.1 (A), TP2.1, U2.37 (PA14)
- new net DAP_SWDIO: JP2.1 (A), TP1.1, U2.34 (PA13)
- new net TRG_NRST: J21.4 (Pin_4)
- new net TRG_RXD: J1.3 (Pin_3), J21.5 (Pin_5), R84.2, U15.7 (A6)
- new net TRG_TXD: J1.2 (Pin_2), J21.6 (Pin_6), R56.2, R85.1, U15.6 (A5)
- no-connect marks 11 -> 17
Other:
- note added: "+5V"
- note added: "1.8V, 3.3V, 5V"
- note added: "DAP_TRG_SCL"
- note added: "DAP_TRG_SDA"
- note added: "JTDI"
- note added: "TXS0108ERGYR"
- note added: "To power page"
- note added: "isolate swd!"
- note added: "pull up?"
- note removed: "Board Ident: PC13 = 0"
- note removed: "JP4"
- title: (none) -> DAPLink
- moved on the sheet: C1, C10, C11, C12, C13, C14, C2, C3, C4, C5, C6, C7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

Commit message: tmp
Parts:
- C11, C12, C14, C6, C7, C9: footprint (none) -> Capacitor_SMD:C_0402_1005Metric
- R1, R10, R11, R12, R13, R14, R15, R16, R17, R18, R19, R2, R21, R22, R23, R24, R25, R26, R3, R4, R5, R56, R6, R7, R8, R84, R85, R9: footprint (none) -> Resistor_SMD:R_0402_1005Metric
Changed lines of the file:
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@@
       (effects (font (size 1.27 1.27)) (justify right))
     )
-    (property "Footprint" "" (at 330.2 192.278 90)
+    (property "Footprint" "Resistor_SMD:R_0402_1005Metric" (at 330.2 192.278 90)
       (effects (font (size 1.27 1.27)) hide)
     )
@@
       (effects (font (size 1.27 1.27)) (justify left))
     )
-    (property "Footprint" "" (at 87.122 171.45 90)
+    (property "Footprint" "Resistor_SMD:R_0402_1005Metric" (at 87.122 171.45 90)
       (effects (font (size 1.27 1.27)) hide)
     )
@@
       (effects (font (size 1.27 1.27)))
     )
-    (property "Footprint" "" (at 196.85 52.578 90)
+    (property "Footprint" "Resistor_SMD:R_0402_1005Metric" (at 196.85 52.578 90)
       (effects (font (size 1.27 1.27)) hide)
     )
@@
       (effects (font (size 1.27 1.27)))
     )
-    (property "Footprint" "" (at 196.85 39.878 90)
+    (property "Footprint" "Resistor_SMD:R_0402_1005Metric" (at 196.85 39.878 90)
       (effects (font (size 1.27 1.27)) hide)
     )
@@
       (effects (font (size 1.27 1.27)) (justify left))
     )
-    (property "Footprint" "" (at 172.212 246.38 90)
+    (property "Footprint" "Resistor_SMD:R_0402_1005Metric" (at 172.212 246.38 90)
       (effects (font (size 1.27 1.27)) hide)
     )
@@
       (effects (font (size 1.27 1.27)) (justify left))
     )
-    (property "Footprint" "" (at 36.322 171.45 90)
+    (property "Footprint" "Resistor_SMD:R_0402_1005Metric" (at 36.322 171.45 90)
       (effects (font (size 1.27 1.27)) hide)
     )
@@
       (effects (font (size 1.27 1.27)) (justify right))
     )
-    (property "Footprint" "" (at 349.25 250.698 90)
+    (property "Footprint" "Resistor_SMD:R_0402_1005Metric" (at 349.25 250.698 90)
       (effects (font (size 1.27 1.27)) hide)
     )
@@
       (effects (font (size 1.27 1.27)) (justify left))
     )
-    (property "Footprint" "" (at 140.6652 86.36 0)
+    (property "Footprint" "Capacitor_SMD:C_0402_1005Metric" (at 140.6652 86.36 0)
       (effects (font (size 1.27 1.27)) hide)
     )
@@
       (effects (font (size 1.27 1.27)))
     )
-    (property "Footprint" "" (at 107.95 103.378 90)
+    (property "Footprint" "Resistor_SMD:R_0402_1005Metric" (at 107.95 103.378 90)
       (effects (font (size 1.27 1.27)) hide)
     )
@@
       (effects (font (size 1.27 1.27)) (justify right))
     )
-    (property "Footprint" "" (at 186.69 231.648 90)
+    (property "Footprint" "Resistor_SMD:R_0402_1005Metric" (at 186.69 231.648 90)
       (effects (font (size 1.27 1.27)) hide)
     )
@@
       (effects (font (size 1.27 1.27)))
     )
-    (property "Footprint" "" (at 196.85 77.978 90)
+    (property "Footprint" "Resistor_SMD:R_0402_1005Metric" (at 196.85 77.978 90)
       (effects (font (size 1.27 1.27)) hide)
     )
@@
       (effects (font (size 1.27 1.27)))
     )
-    (property "Footprint" "" (at 107.95 109.728 90)
+    (property "Footprint" "Resistor_SMD:R_0402_1005Metric" (at 107.95 109.728 90)
       (effects (font (size 1.27 1.27)) hide)
     )
@@
       (effects (font (size 1.27 1.27)) (justify left))
     )
-    (property "Footprint" "" (at 87.122 184.15 90)
+    (property "Footprint" "Resistor_SMD:R_0402_1005Metric" (at 87.122 184.15 90)
       (effects (font (size 1.27 1.27)) hide)
     )
@@
       (effects (font (size 1.27 1.27)))
     )
-    (property "Footprint" "" (at 361.95 169.418 90)
+    (property "Footprint" "Resistor_SMD:R_0402_1005Metric" (at 361.95 169.418 90)
       (effects (font (size 1.27 1.27)) hide)
     )
@@
       (effects (font (size 1.27 1.27)) (justify right))
     )
-    (property "Footprint" "" (at 198.12 216.408 90)
+    (property "Footprint" "Resistor_SMD:R_0402_1005Metric" (at 198.12 216.408 90)
       (effects (font (size 1.27 1.27)) hide)
     )
@@
       (effects (font (size 1.27 1.27)) (justify left))
     )
-    (property "Footprint" "" (at 112.522 184.15 90)
+    (property "Footprint" "Resistor_SMD:R_0402_1005Metric" (at 112.522 184.15 90)
       (effects (font (size 1.27 1.27)) hide)
     )
@@
       (effects (font (size 1.27 1.27)) (justify left))
     )
-    (property "Footprint" "" (at 61.722 184.15 90)
+    (property "Footprint" "Resistor_SMD:R_0402_1005Metric" (at 61.722 184.15 90)
       (effects (font (size 1.27 1.27)) hide)
     )
@@
       (effects (font (size 1.27 1.27)) (justify right))
     )
-    (property "Footprint" "" (at 330.2 189.738 90)
+    (property "Footprint" "Resistor_SMD:R_0402_1005Metric" (at 330.2 189.738 90)
       (effects (font (size 1.27 1.27)) hide)
     )
@@
       (effects (font (size 1.27 1.27)) (justify left))
     )
-    (property "Footprint" "" (at 204.1652 86.36 0)
+    (property "Footprint" "Capacitor_SMD:C_0402_1005Metric" (at 204.1652 86.36 0)
       (effects (font (size 1.27 1.27)) hide)
     )
@@
       (effects (font (size 1.27 1.27)) (justify right))
     )
-    (property "Footprint" "" (at 186.69 241.808 90)
+    (property "Footprint" "Resistor_SMD:R_0402_1005Metric" (at 186.69 241.808 90)
       (effects (font (size 1.27 1.27)) hide)
     )
@@
       (effects (font (size 1.27 1.27)))
     )
-    (property "Footprint" "" (at 243.84 239.268 90)
+    (property "Footprint" "Resistor_SMD:R_0402_1005Metric" (at 243.84 239.268 90)
       (effects (font (size 1.27 1.27)) hide)
     )
@@
       (effects (font (size 1.27 1.27)) (justify left))
     )
-    (property "Footprint" "" (at 353.822 173.99 90)
+    (property "Footprint" "Resistor_SMD:R_0402_1005Metric" (at 353.822 173.99 90)
       (effects (font (size 1.27 1.27)) hide)
     )
@@
       (effects (font (size 1.27 1.27)) (justify left))
     )
-    (property "Footprint" "" (at 326.0852 17.78 0)
+    (property "Footprint" "Capacitor_SMD:C_0402_1005Metric" (at 326.0852 17.78 0)
       (effects (font (size 1.27 1.27)) hide)
     )
@@
       (effects (font (size 1.27 1.27)) (justify left))
     )
-    (property "Footprint" "" (at 353.822 161.29 90)
+    (property "Footprint" "Resistor_SMD:R_0402_1005Metric" (at 353.822 161.29 90)
       (effects (font (size 1.27 1.27)) hide)
     )
@@
       (effects (font (size 1.27 1.27)) (justify right))
     )
-    (property "Footprint" "" (at 186.69 236.728 90)
+    (property "Footprint" "Resistor_SMD:R_0402_1005Metric" (at 186.69 236.728 90)
       (effects (font (size 1.27 1.27)) hide)
     )
@@
       (effects (font (size 1.27 1.27)) (justify right))
     )
-    (property "Footprint" "" (at 330.2 187.198 90)
+    (property "Footprint" "Resistor_SMD:R_0402_1005Metric" (at 330.2 187.198 90)
       (effects (font (size 1.27 1.27)) hide)
     )
@@
       (effects (font (size 1.27 1.27)) (justify left))
     )
-    (property "Footprint" "" (at 127.9652 86.36 0)
+    (property "Footprint" "Capacitor_SMD:C_0402_1005Metric" (at 127.9652 86.36 0)
       (effects (font (size 1.27 1.27)) hide)
     )
@@
       (effects (font (size 1.27 1.27)))
     )
-    (property "Footprint" "" (at 50.8 141.478 90)
+    (property "Footprint" "Resistor_SMD:R_0402_1005Metric" (at 50.8 141.478 90)
       (effects (font (size 1.27 1.27)) hide)
     )
@@
       (effects (font (size 1.27 1.27)) (justify right))
     )
-    (property "Footprint" "" (at 330.2 184.658 90)
+    (property "Footprint" "Resistor_SMD:R_0402_1005Metric" (at 330.2 184.658 90)
       (effects (font (size 1.27 1.27)) hide)
     )
@@
       (effects (font (size 1.27 1.27)) (justify left))
     )
-    (property "Footprint" "" (at 376.8852 17.78 0)
+    (property "Footprint" "Capacitor_SMD:C_0402_1005Metric" (at 376.8852 17.78 0)
       (effects (font (size 1.27 1.27)) hide)
     )
@@
       (effects (font (size 1.27 1.27)) (justify left))
     )
-    (property "Footprint" "" (at 367.9952 17.78 0)
+    (property "Footprint" "Capacitor_SMD:C_0402_1005Metric" (at 367.9952 17.78 0)
       (effects (font (size 1.27 1.27)) hide)
     )
@@
       (effects (font (size 1.27 1.27)))
     )
-    (property "Footprint" "" (at 260.35 281.178 90)
+    (property "Footprint" "Resistor_SMD:R_0402_1005Metric" (at 260.35 281.178 90)
       (effects (font (size 1.27 1.27)) hide)
     )
@@
       (effects (font (size 1.27 1.27)) (justify left))
     )
-    (property "Footprint" "" (at 112.522 171.45 90)
+    (property "Footprint" "Resistor_SMD:R_0402_1005Metric" (at 112.522 171.45 90)
       (effects (font (size 1.27 1.27)) hide)
     )
@@
       (effects (font (size 1.27 1.27)))
     )
-    (property "Footprint" "" (at 260.35 283.718 90)
-      (effects (font (size 1.27 1.27)) hide)
-    )
+    (property "Footprint" "Resistor_SMD:R_0402_1005Metric" (at 260.35 283.718 90)
+      (effects (font (size 1.27 1.27)) hide)
+    )
