File: prototype/hub.kicad_sch (KiCad schematic)
At the start: 2 parts, among them U1 LAN9514I-JZX, Y1 Crystal_GND23

Commit message: nrf5240
Parts:
- added C74, C75: 33p, symbol Device:C
- added C80 (x4): 15p, Capacitor_SMD:C_0603_1608Metric, symbol Device:C
- added C80: 22n, Capacitor_SMD:C_0603_1608Metric, symbol Device:C
- added C? (x16): 0.1u, symbol Device:C
- added C?: 1u, symbol Device:C
- added C?: 4.7u, symbol Device:C
- added D10, D11, D12, D9: LED, symbol Device:LED
- added J10: HR911105A, Connector_RJ:RJ45_Hanrun_HR911105A, symbol Connector:RJ45_LED
- added J6: 622002115121, symbol Connector_Generic:Conn_01x02
- added L5 (x2): 120@2.0A, symbol Device:L
- added R32: 12k, symbol Device:R
- added R69 (x4): 49.9, Resistor_SMD:R_0603_1608Metric, symbol Device:R
- added R71: 10, Resistor_SMD:R_0603_1608Metric, symbol Device:R
- added R72, R73: 330, Resistor_SMD:R_0603_1608Metric, symbol Device:R
- added R73: 0, Resistor_SMD:R_1206_3216Metric, symbol Device:R
- added R75: 1M, symbol Device:R
- added R79: 12.4k, symbol Device:R
- added R80: 10k, symbol Device:R
- added SW2, SW3, SW4, SW5: SW_Push_SPDT, symbol Switch:SW_Push_SPDT
- added Y2: 25MHz, symbol Device:Crystal_GND24
Connections:
- net GND: now also U1.34 (TEST2), U1.44 (CLK24_EN), C74.2, C75.2, C80.2, C80.2, C80.2, C80.2, C80.2, C?.2, C?.2, C?.2, C?.2, C?.2, C?.2, C?.2, C?.2, C?.2, C?.2, C?.2, C?.2, C?.2, C?.2, C?.2, C?.2, C?.2, C?.2, R32.2, R73.1, R79.2, Y2.2, Y2.4
- net HUB_RX_N: now also C80.1, J10.6, R69.2
- net HUB_TX_N: now also C80.1, J10.3, R69.2
- net HUB_TX_P: now also C80.1, J10.1, R69.2
- net VDD33A: now reaches U1.10 (VDD33A), U1.49 (VDD33A), U1.5 (VDD33A), U1.51 (VDD33A), U1.54 (VDD33A), U1.57 (VDD33A), U1.64 (VDD33A)
- net VDD33A: now also C?.1, C?.1, C?.1, C?.1, C?.1, C?.1, C?.1, L5.1, R69.1, R69.1, R69.1, R69.1, R71.1
- net at U1.12 (~{RESET}): now also C?.1, R80.2
- net VDD18CORE: now reaches U1.15 (VDD18CORE), U1.38 (VDD18CORE)
- net VDD18CORE: now also C?.1, C?.1, C?.1
- net VDD33IO: now reaches U1.19 (VDD33IO), U1.27 (VDD33IO), U1.33 (VDD33IO), U1.39 (VDD33IO), U1.46 (VDD33IO)
- net VDD33IO: now also U1.11 (VBUS_DET), U1.28 (~{TRST}), U1.29 (TMS), U1.30 (TDI), U1.32 (TCK), U1.40 (TEST3), C?.1, C?.1, C?.1, C?.1, C?.1, J10.10, J10.12, L5.2, R80.1
- net FDX_LED: now reaches U1.20 (~{FDX_LED}/GPIO0)
- net FDX_LED: now also R72.1
- net LNKA_LED: now reaches U1.21 (~{LNKA_LED}/GPIO1)
- net LNKA_LED: now also R73.1
- net EECLK: now reaches U1.23 (EECLK)
- net EECS: now reaches U1.24 (EECS)
- net EEDO: now reaches U1.25 (EEDO)
- net EEDI: now reaches U1.26 (EEDI)
- net VDD18ETHPLL: now reaches U1.48 (VDD18ETHPLL)
- net VDD18ETHPLL: now also C?.1, L5.1
- net HUB_XO: now reaches U1.60 (XO)
- net HUB_XO: now also C74.1, R75.2, Y2.1
- net HUB_XI: now reaches U1.61 (XI)
- net HUB_XI: now also C75.1, R75.1, Y2.3
- net VDD18USBPLL: now reaches U1.62 (VDD18USBPLL)
- net VDD18USBPLL: now also C?.1, L5.2
- net +3.3V: now reaches U1.41 (AUTOMDIX_EN)
- net at U1.50 (EXRES): now also R79.1
- net HUB_USB_N: now reaches U1.58 (USBDM0)
- net HUB_USB_P: now reaches U1.59 (USBDP0)
- net at U1.63 (USBRBIAS): now also R32.1
- new net: J10.11, R72.2
- new net: C80.1, J10.2, J10.5, R71.2
- new net: J10.9, R73.2
- new net Earth: J10.8, R73.2
- new net HUB_RX_P: C80.1, J10.4, R69.2
- no-connect marks 0 -> 11
Other:
- note added: "622002115121"
- note added: "check it"
- note added: "to S76S"

Commit message: DAPLink, FT2232H
Parts:
- removed Y1: Crystal_GND23, symbol Device:Crystal_GND23
- added C?: 0.1u, symbol Device:C
- added F1: Fuse, symbol Device:Fuse
- added FB1: 0603, symbol Device:FerriteBead_Small
- added J9: USB_A, symbol Connector:USB_A
- added P1: USB_C_Plug_USB2.0, symbol Connector:USB_C_Plug_USB2.0
- added U23: TS3USB30ERSW, Package_DFN_QFN:UQFN-10_1.4x1.8mm_P0.4mm, symbol chrns_ic_connectivity:TS3USB30ERSW
- added U9: USBLC6-4SC6, Package_TO_SOT_SMD:SOT-23-6, symbol Power_Protection:USBLC6-4SC6
- J10: Part number (none) -> HR911105A; PartNumber HR911105A -> (none)
- J6: digikey 732-13627-ND -> (none)
Connections:
- net +3.3V: now also C?.1, U23.9 (VCC)
- net GND: now also C?.2, J9.4 (GND), J9.5 (Shield), U23.4 (GND), U23.8 (~{OE}), U9.2 (GND)
- net DAP_USB_D_N: now reaches U1.1 (USBDM2)
- net DAP_USB_D_P: now reaches U1.2 (USBDP2)
- net NRF_USB_D_P: now reaches U1.3 (USBDM3)
- net NRF_USB_D_N: now reaches U1.4 (USBDP3)
- net CY_USB_D_N: now reaches U1.6 (USBDM4)
- net CY_USB_D_P: now reaches U1.7 (USBDP4)
- net HUB_SW_D_N: now reaches U1.8 (USBDM5)
- net HUB_SW_D_N: now also U23.5 (D-)
- net HUB_SW_D_P: now reaches U1.9 (USBDP5)
- net HUB_SW_D_P: now also U23.3 (D+)
- new net: F1.2, FB1.1, U9.5 (VBUS)
- new net: P1.A1 (GND), P1.A12 (GND), P1.B1 (GND), P1.B12 (GND)
- new net: P1.A4 (VBUS), P1.A9 (VBUS), P1.B4 (VBUS), P1.B9 (VBUS)
- new net: F1.1, J9.1 (VBUS)
- new net 3V3_VBUS: FB1.2
- new net EXT_D_N: J9.2 (D-), U23.6 (D2-), U9.1 (I/O1)
- new net EXT_D_P: J9.3 (D+), U23.2 (D2+), U9.4 (I/O3)
- new net FT_USB_D_N: U23.7 (D1-)
- new net FT_USB_D_P: U23.1 (D1+)
- no-connect marks 11 -> 13

Commit message: tmp
Parts:
- removed F1: Fuse, symbol Device:Fuse
- removed FB1: 0603, symbol Device:FerriteBead_Small
- removed J9: USB_A, symbol Connector:USB_A
- removed P1: USB_C_Plug_USB2.0, symbol Connector:USB_C_Plug_USB2.0
- removed U9: USBLC6-4SC6, Package_TO_SOT_SMD:SOT-23-6, symbol Power_Protection:USBLC6-4SC6
Connections:
- no-connect marks 13 -> 11

Commit message: tmp
Parts:
- C74, C75, C? (x19): footprint (none) -> Capacitor_SMD:C_0402_1005Metric
- R32, R75, R79, R80: footprint (none) -> Resistor_SMD:R_0402_1005Metric
Changed lines of the file:
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@@
       (effects (font (size 1.27 1.27)) (justify left))
     )
-    (property "Footprint" "" (at 83.5152 187.96 0)
+    (property "Footprint" "Capacitor_SMD:C_0402_1005Metric" (at 83.5152 187.96 0)
       (effects (font (size 1.27 1.27)) hide)
     )
@@
       (effects (font (size 1.27 1.27)) (justify left))
     )
-    (property "Footprint" "" (at 102.5652 187.96 0)
+    (property "Footprint" "Capacitor_SMD:C_0402_1005Metric" (at 102.5652 187.96 0)
       (effects (font (size 1.27 1.27)) hide)
     )
@@
       (effects (font (size 1.27 1.27)) (justify left))
     )
-    (property "Footprint" "" (at 201.422 85.09 90)
+    (property "Footprint" "Resistor_SMD:R_0402_1005Metric" (at 201.422 85.09 90)
       (effects (font (size 1.27 1.27)) hide)
     )
@@
       (effects (font (size 1.27 1.27)) (justify left))
     )
-    (property "Footprint" "" (at 163.5252 187.96 0)
+    (property "Footprint" "Capacitor_SMD:C_0402_1005Metric" (at 163.5252 187.96 0)
       (effects (font (size 1.27 1.27)) hide)
     )
@@
       (effects (font (size 1.27 1.27)) (justify left))
     )
-    (property "Footprint" "" (at 23.622 60.96 90)
+    (property "Footprint" "Resistor_SMD:R_0402_1005Metric" (at 23.622 60.96 90)
       (effects (font (size 1.27 1.27)) hide)
     )
@@
       (effects (font (size 1.27 1.27)) (justify left))
     )
-    (property "Footprint" "" (at 32.7152 187.96 0)
+    (property "Footprint" "Capacitor_SMD:C_0402_1005Metric" (at 32.7152 187.96 0)
       (effects (font (size 1.27 1.27)) hide)
     )
@@
       (effects (font (size 1.27 1.27)) (justify left))
     )
-    (property "Footprint" "" (at 101.092 133.35 90)
+    (property "Footprint" "Resistor_SMD:R_0402_1005Metric" (at 101.092 133.35 90)
       (effects (font (size 1.27 1.27)) hide)
     )
@@
       (effects (font (size 1.27 1.27)) (justify left))
     )
-    (property "Footprint" "" (at 26.3652 74.93 0)
+    (property "Footprint" "Capacitor_SMD:C_0402_1005Metric" (at 26.3652 74.93 0)
       (effects (font (size 1.27 1.27)) hide)
     )
@@
       (effects (font (size 1.27 1.27)) (justify left))
     )
-    (property "Footprint" "" (at 77.1652 187.96 0)
+    (property "Footprint" "Capacitor_SMD:C_0402_1005Metric" (at 77.1652 187.96 0)
       (effects (font (size 1.27 1.27)) hide)
     )
@@
       (effects (font (size 1.27 1.27)) (justify left))
     )
-    (property "Footprint" "" (at 89.8652 187.96 0)
+    (property "Footprint" "Capacitor_SMD:C_0402_1005Metric" (at 89.8652 187.96 0)
       (effects (font (size 1.27 1.27)) hide)
     )
@@
       (effects (font (size 1.27 1.27)) (justify left))
     )
-    (property "Footprint" "" (at 115.2652 187.96 0)
+    (property "Footprint" "Capacitor_SMD:C_0402_1005Metric" (at 115.2652 187.96 0)
       (effects (font (size 1.27 1.27)) hide)
     )
@@
       (effects (font (size 1.27 1.27)) (justify left))
     )
-    (property "Footprint" "" (at 45.4152 187.96 0)
+    (property "Footprint" "Capacitor_SMD:C_0402_1005Metric" (at 45.4152 187.96 0)
       (effects (font (size 1.27 1.27)) hide)
     )
@@
       (effects (font (size 1.27 1.27)) (justify left))
     )
-    (property "Footprint" "" (at 39.0652 187.96 0)
+    (property "Footprint" "Capacitor_SMD:C_0402_1005Metric" (at 39.0652 187.96 0)
       (effects (font (size 1.27 1.27)) hide)
     )
@@
       (effects (font (size 1.27 1.27)) (justify left))
     )
-    (property "Footprint" "" (at 51.7652 245.11 0)
+    (property "Footprint" "Capacitor_SMD:C_0402_1005Metric" (at 51.7652 245.11 0)
       (effects (font (size 1.27 1.27)) hide)
     )
@@
       (effects (font (size 1.27 1.27)) (justify left))
     )
-    (property "Footprint" "" (at 58.1152 187.96 0)
+    (property "Footprint" "Capacitor_SMD:C_0402_1005Metric" (at 58.1152 187.96 0)
       (effects (font (size 1.27 1.27)) hide)
     )
@@
       (effects (font (size 1.27 1.27)) (justify left))
     )
-    (property "Footprint" "" (at 64.4652 187.96 0)
+    (property "Footprint" "Capacitor_SMD:C_0402_1005Metric" (at 64.4652 187.96 0)
       (effects (font (size 1.27 1.27)) hide)
     )
@@
       (effects (font (size 1.27 1.27)) (justify left))
     )
-    (property "Footprint" "" (at 103.8352 149.86 0)
+    (property "Footprint" "Capacitor_SMD:C_0402_1005Metric" (at 103.8352 149.86 0)
       (effects (font (size 1.27 1.27)) hide)
     )
@@
       (effects (font (size 1.27 1.27)) (justify left))
     )
-    (property "Footprint" "" (at 127.9652 187.96 0)
+    (property "Footprint" "Capacitor_SMD:C_0402_1005Metric" (at 127.9652 187.96 0)
       (effects (font (size 1.27 1.27)) hide)
     )
@@
       (effects (font (size 1.27 1.27)) (justify left))
     )
-    (property "Footprint" "" (at 121.6152 187.96 0)
+    (property "Footprint" "Capacitor_SMD:C_0402_1005Metric" (at 121.6152 187.96 0)
       (effects (font (size 1.27 1.27)) hide)
     )
@@
       (effects (font (size 1.27 1.27)) (justify left))
     )
-    (property "Footprint" "" (at 150.8252 187.96 0)
+    (property "Footprint" "Capacitor_SMD:C_0402_1005Metric" (at 150.8252 187.96 0)
       (effects (font (size 1.27 1.27)) hide)
     )
@@
       (effects (font (size 1.27 1.27)) (justify left))
     )
-    (property "Footprint" "" (at 51.7652 187.96 0)
+    (property "Footprint" "Capacitor_SMD:C_0402_1005Metric" (at 51.7652 187.96 0)
       (effects (font (size 1.27 1.27)) hide)
     )
@@
       (effects (font (size 1.27 1.27)) (justify left))
     )
-    (property "Footprint" "" (at 96.2152 187.96 0)
+    (property "Footprint" "Capacitor_SMD:C_0402_1005Metric" (at 96.2152 187.96 0)
       (effects (font (size 1.27 1.27)) hide)
     )
@@
       (effects (font (size 1.27 1.27)) (justify left))
     )
-    (property "Footprint" "" (at 201.422 111.76 90)
+    (property "Footprint" "Resistor_SMD:R_0402_1005Metric" (at 201.422 111.76 90)
       (effects (font (size 1.27 1.27)) hide)
     )
@@
       (effects (font (size 1.27 1.27)) (justify left))
     )
-    (property "Footprint" "" (at 26.3652 187.96 0)
+    (property "Footprint" "Capacitor_SMD:C_0402_1005Metric" (at 26.3652 187.96 0)
       (effects (font (size 1.27 1.27)) hide)
     )
@@
       (effects (font (size 1.27 1.27)) (justify left))
     )
-    (property "Footprint" "" (at 119.0752 149.86 0)
-      (effects (font (size 1.27 1.27)) hide)
-    )
+    (property "Footprint" "Capacitor_SMD:C_0402_1005Metric" (at 119.0752 149.86 0)
+      (effects (font (size 1.27 1.27)) hide)
+    )
