File: prototype/logic.kicad_sch (KiCad schematic)
At the start: 34 parts, among them J4 LOGIC, U5 CY7C68013A-56LTX, U7 24LC00, Y3 24MHz

Commit message: DAPLink, FT2232H
Parts:
- added U15: TXS0108ERGYR, Package_SO:TSSOP-20_4.4x6.5mm_P0.65mm, symbol Logic_LevelTranslator:TXS0108EPW
Connections:
- net CY_USB_D_P: no longer U5.9 (D-)
- net GND: now also U15.11 (GND)
- net LOGIC_CH0: now also U15.1 (A1)
- net LOGIC_CH1: now also U15.3 (A2)
- net LOGIC_CH2: now also U15.4 (A3)
- net LOGIC_CH3: now also U15.5 (A4)
- net LOGIC_CH4: now also U15.6 (A5)
- net LOGIC_CH5: now also U15.7 (A6)
- net LOGIC_CH6: now also U15.8 (A7)
- net LOGIC_CH7: now also U15.9 (A8)
- new net 3V3_FT: U15.10 (OE), U15.2 (VCCA)
- new net CH0: U15.20 (B1)
- new net CH1: U15.18 (B2)
- new net CH2: U15.17 (B3)
- new net CH3: U15.16 (B4)
- new net CH4: U15.15 (B5)
- new net CH5: U15.14 (B6)
- new net CH6: U15.13 (B7)
- new net CH7: U15.12 (B8)
- new net CY_USB_D_N: U5.9 (D-)
Other:
- note added: "1.8V, 3.3V, 5V"
- note added: "TXS0108ERGYR"

Commit message: tmp
Connections:
- net 3V3_FT is gone; now on net 3V3_LOGIC: U15.10 (OE), U15.2 (VCCA)
- net 3V3LOGIC renamed 3V3_LOGIC
Changed lines of the file:
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@@
     (effects (font (size 1.524 1.524)) (justify left bottom))
-  )
-  (label "3V3LOGIC" (at 256.54 214.63 0) (fields_autoplaced)
-    (effects (font (size 1.27 1.27)) (justify left bottom))
   )
   (label "LOGIC_CH1" (at 279.4 50.8 180) (fields_autoplaced)
     (effects (font (size 1.524 1.524)) (justify right bottom))
   )
+  (label "3V3_LOGIC" (at 180.34 214.63 0) (fields_autoplaced)
+    (effects (font (size 1.27 1.27)) (justify left bottom))
+  )
   (label "LOGIC_CH4" (at 298.45 35.56 0) (fields_autoplaced)
     (effects (font (size 1.524 1.524)) (justify left bottom))
@@
     (effects (font (size 1.524 1.524)) (justify right bottom))
   )
-  (label "3V3LOGIC" (at 139.7 25.4 180) (fields_autoplaced)
-    (effects (font (size 1.27 1.27)) (justify right bottom))
-  )
   (label "LOGIC_CH4" (at 241.3 55.88 0) (fields_autoplaced)
     (effects (font (size 1.524 1.524)) (justify left bottom))
@@
     (effects (font (size 1.524 1.524)) (justify right bottom))
   )
-  (label "3V3LOGIC" (at 303.53 113.03 0) (fields_autoplaced)
+  (label "3V3_LOGIC" (at 256.54 214.63 0) (fields_autoplaced)
     (effects (font (size 1.27 1.27)) (justify left bottom))
   )
@@
     (effects (font (size 1.524 1.524)) (justify left bottom))
   )
+  (label "3V3_LOGIC" (at 107.95 71.12 180) (fields_autoplaced)
+    (effects (font (size 1.27 1.27)) (justify right bottom))
+  )
   (label "CH4" (at 342.9 35.56 180) (fields_autoplaced)
     (effects (font (size 1.524 1.524)) (justify right bottom))
   )
+  (label "3V3_LOGIC" (at 139.7 25.4 180) (fields_autoplaced)
+    (effects (font (size 1.27 1.27)) (justify right bottom))
+  )
   (label "CY_CH3" (at 139.7 48.26 180) (fields_autoplaced)
     (effects (font (size 1.524 1.524)) (justify right bottom))
   )
+  (label "3V3_LOGIC" (at 354.33 110.49 0) (fields_autoplaced)
+    (effects (font (size 1.27 1.27)) (justify left bottom))
+  )
   (label "LOGIC_CH7" (at 279.4 58.42 180) (fields_autoplaced)
     (effects (font (size 1.524 1.524)) (justify right bottom))
@@
     (effects (font (size 1.524 1.524)) (justify right bottom))
   )
-  (label "3V3LOGIC" (at 107.95 111.76 180) (fields_autoplaced)
-    (effects (font (size 1.27 1.27)) (justify right bottom))
-  )
   (label "xCLK" (at 271.78 63.5 0) (fields_autoplaced)
     (effects (font (size 1.524 1.524)) (justify left bottom))
@@
     (effects (font (size 1.524 1.524)) (justify right bottom))
   )
-  (label "3V3LOGIC" (at 254 91.44 0) (fields_autoplaced)
-    (effects (font (size 1.27 1.27)) (justify left bottom))
-  )
   (label "~{RESET}" (at 19.05 78.74 0) (fields_autoplaced)
     (effects (font (size 1.524 1.524)) (justify left bottom))
@@
     (effects (font (size 1.524 1.524)) (justify right bottom))
   )
-  (label "3V3LOGIC" (at 50.8 30.48 180) (fields_autoplaced)
+  (label "3V3_LOGIC" (at 50.8 30.48 180) (fields_autoplaced)
     (effects (font (size 1.27 1.27)) (justify right bottom))
   )
@@
     (effects (font (size 1.27 1.27)) (justify left bottom))
   )
-  (label "3V3LOGIC" (at 180.34 214.63 0) (fields_autoplaced)
-    (effects (font (size 1.27 1.27)) (justify left bottom))
-  )
   (label "CY_CH0" (at 139.7 40.64 180) (fields_autoplaced)
     (effects (font (size 1.524 1.524)) (justify right bottom))
@@
     (effects (font (size 1.524 1.524)) (justify left bottom))
   )
-  (label "3V3LOGIC" (at 228.6 95.25 0) (fields_autoplaced)
-    (effects (font (size 1.27 1.27)) (justify left bottom))
-  )
-  (label "3V3_FT" (at 304.8 12.7 0) (fields_autoplaced)
-    (effects (font (size 1.27 1.27)) (justify left bottom))
-  )
   (label "LOGIC_CH2" (at 241.3 53.34 0) (fields_autoplaced)
     (effects (font (size 1.524 1.524)) (justify left bottom))
@@
     (effects (font (size 1.524 1.524)) (justify right bottom))
   )
+  (label "3V3_LOGIC" (at 228.6 95.25 180) (fields_autoplaced)
+    (effects (font (size 1.27 1.27)) (justify right bottom))
+  )
   (label "LOGIC_CH2" (at 298.45 30.48 0) (fields_autoplaced)
     (effects (font (size 1.524 1.524)) (justify left bottom))
@@
     (effects (font (size 1.524 1.524)) (justify right bottom))
   )
+  (label "3V3_LOGIC" (at 107.95 111.76 180) (fields_autoplaced)
+    (effects (font (size 1.27 1.27)) (justify right bottom))
+  )
   (label "CY_RDY1" (at 107.95 86.36 180) (fields_autoplaced)
     (effects (font (size 1.27 1.27)) (justify right bottom))
@@
     (effects (font (size 1.524 1.524)) (justify left bottom))
   )
+  (label "3V3_LOGIC" (at 303.53 113.03 0) (fields_autoplaced)
+    (effects (font (size 1.27 1.27)) (justify left bottom))
+  )
   (label "CY_SCL" (at 273.05 99.06 180) (fields_autoplaced)
     (effects (font (size 1.27 1.27)) (justify right bottom))
   )
+  (label "3V3_LOGIC" (at 254 91.44 180) (fields_autoplaced)
+    (effects (font (size 1.27 1.27)) (justify right bottom))
+  )
   (label "CY_CH5" (at 139.7 53.34 180) (fields_autoplaced)
     (effects (font (size 1.524 1.524)) (justify right bottom))
@@
     (effects (font (size 1.27 1.27)) (justify left bottom))
   )
-  (label "3V3LOGIC" (at 107.95 71.12 180) (fields_autoplaced)
-    (effects (font (size 1.27 1.27)) (justify right bottom))
-  )
   (label "IFCLK" (at 76.2 91.44 180) (fields_autoplaced)
     (effects (font (size 1.27 1.27)) (justify right bottom))
   )
+  (label "3V3_LOGIC" (at 304.8 12.7 0) (fields_autoplaced)
+    (effects (font (size 1.27 1.27)) (justify left bottom))
+  )
   (label "xTRIG" (at 248.92 63.5 180) (fields_autoplaced)
     (effects (font (size 1.524 1.524)) (justify right bottom))
@@
     (effects (font (size 1.524 1.524)) (justify right bottom))
   )
-  (label "3V3LOGIC" (at 354.33 110.49 0) (fields_autoplaced)
-    (effects (font (size 1.27 1.27)) (justify left bottom))
+  (hierarchical_label "3V3_LOGIC" (shape input) (at 50.8 30.48 0) (fields_autoplaced)
+    (effects (font (size 1.27 1.27)) (justify left))
   )
   (hierarchical_label "CY_USB_D_P" (shape bidirectional) (at 30.48 93.98 180) (fields_autoplaced)

Commit message: tmp
Parts:
- C15, C16, C17, C18, C19, C20, C21, C22, C23, C24, C25, C26, C27, C28: footprint (none) -> Capacitor_SMD:C_0402_1005Metric
- R20, R27, R28, R29, R30, R31, R32, R33, R34, R35, R36, R37, R38, R41, R42: footprint (none) -> Resistor_SMD:R_0402_1005Metric
Changed lines of the file:
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@@
       (effects (font (size 1.27 1.27)) (justify left))
     )
-    (property "Footprint" "" (at 87.122 77.47 90)
+    (property "Footprint" "Resistor_SMD:R_0402_1005Metric" (at 87.122 77.47 90)
       (effects (font (size 1.27 1.27)) hide)
     )
@@
       (effects (font (size 1.27 1.27)) (justify left))
     )
-    (property "Footprint" "" (at 112.522 31.75 90)
+    (property "Footprint" "Resistor_SMD:R_0402_1005Metric" (at 112.522 31.75 90)
       (effects (font (size 1.27 1.27)) hide)
     )
@@
       (effects (font (size 1.27 1.27)) (justify left))
     )
-    (property "Footprint" "" (at 74.422 31.75 90)
+    (property "Footprint" "Resistor_SMD:R_0402_1005Metric" (at 74.422 31.75 90)
       (effects (font (size 1.27 1.27)) hide)
     )
@@
       (effects (font (size 1.27 1.27)) (justify left))
     )
-    (property "Footprint" "" (at 102.5652 175.26 0)
+    (property "Footprint" "Capacitor_SMD:C_0402_1005Metric" (at 102.5652 175.26 0)
       (effects (font (size 1.27 1.27)) hide)
     )
@@
       (effects (font (size 1.27 1.27)) (justify left))
     )
-    (property "Footprint" "" (at 244.8052 227.33 0)
+    (property "Footprint" "Capacitor_SMD:C_0402_1005Metric" (at 244.8052 227.33 0)
       (effects (font (size 1.27 1.27)) hide)
     )
@@
       (effects (font (size 1.27 1.27)) (justify left))
     )
-    (property "Footprint" "" (at 355.2952 135.89 0)
+    (property "Footprint" "Capacitor_SMD:C_0402_1005Metric" (at 355.2952 135.89 0)
       (effects (font (size 1.27 1.27)) hide)
     )
@@
       (effects (font (size 1.27 1.27)) (justify left))
     )
-    (property "Footprint" "" (at 80.772 31.75 90)
+    (property "Footprint" "Resistor_SMD:R_0402_1005Metric" (at 80.772 31.75 90)
       (effects (font (size 1.27 1.27)) hide)
     )
@@
       (effects (font (size 1.27 1.27)) (justify left))
     )
-    (property "Footprint" "" (at 232.1052 227.33 0)
+    (property "Footprint" "Capacitor_SMD:C_0402_1005Metric" (at 232.1052 227.33 0)
       (effects (font (size 1.27 1.27)) hide)
     )
@@
       (effects (font (size 1.27 1.27)) (justify left))
     )
-    (property "Footprint" "" (at 327.152 119.38 90)
+    (property "Footprint" "Resistor_SMD:R_0402_1005Metric" (at 327.152 119.38 90)
       (effects (font (size 1.27 1.27)) hide)
     )
@@
       (effects (font (size 1.27 1.27)) (justify left))
     )
-    (property "Footprint" "" (at 87.122 31.75 90)
+    (property "Footprint" "Resistor_SMD:R_0402_1005Metric" (at 87.122 31.75 90)
       (effects (font (size 1.27 1.27)) hide)
     )
@@
       (effects (font (size 1.27 1.27)) (justify left))
     )
-    (property "Footprint" "" (at 106.172 31.75 90)
+    (property "Footprint" "Resistor_SMD:R_0402_1005Metric" (at 106.172 31.75 90)
       (effects (font (size 1.27 1.27)) hide)
     )
@@
       (effects (font (size 1.27 1.27)) (justify left))
     )
-    (property "Footprint" "" (at 229.5652 105.41 0)
+    (property "Footprint" "Capacitor_SMD:C_0402_1005Metric" (at 229.5652 105.41 0)
       (effects (font (size 1.27 1.27)) hide)
     )
@@
       (effects (font (size 1.27 1.27)) (justify left))
     )
-    (property "Footprint" "" (at 181.3052 227.33 0)
+    (property "Footprint" "Capacitor_SMD:C_0402_1005Metric" (at 181.3052 227.33 0)
       (effects (font (size 1.27 1.27)) hide)
     )
@@
       (effects (font (size 1.27 1.27)) (justify left))
     )
-    (property "Footprint" "" (at 194.0052 227.33 0)
+    (property "Footprint" "Capacitor_SMD:C_0402_1005Metric" (at 194.0052 227.33 0)
       (effects (font (size 1.27 1.27)) hide)
     )
@@
       (effects (font (size 1.27 1.27)) (justify left))
     )
-    (property "Footprint" "" (at 257.5052 227.33 0)
+    (property "Footprint" "Capacitor_SMD:C_0402_1005Metric" (at 257.5052 227.33 0)
       (effects (font (size 1.27 1.27)) hide)
     )
@@
       (effects (font (size 1.27 1.27)) (justify left))
     )
-    (property "Footprint" "" (at 127.9652 175.26 0)
+    (property "Footprint" "Capacitor_SMD:C_0402_1005Metric" (at 127.9652 175.26 0)
       (effects (font (size 1.27 1.27)) hide)
     )
@@
       (effects (font (size 1.27 1.27)) (justify left))
     )
-    (property "Footprint" "" (at 219.4052 227.33 0)
+    (property "Footprint" "Capacitor_SMD:C_0402_1005Metric" (at 219.4052 227.33 0)
       (effects (font (size 1.27 1.27)) hide)
     )
@@
       (effects (font (size 1.27 1.27)) (justify left))
     )
-    (property "Footprint" "" (at 270.2052 227.33 0)
+    (property "Footprint" "Capacitor_SMD:C_0402_1005Metric" (at 270.2052 227.33 0)
       (effects (font (size 1.27 1.27)) hide)
     )
@@
       (effects (font (size 1.27 1.27)) (justify left))
     )
-    (property "Footprint" "" (at 93.472 31.75 90)
+    (property "Footprint" "Resistor_SMD:R_0402_1005Metric" (at 93.472 31.75 90)
       (effects (font (size 1.27 1.27)) hide)
     )
@@
       (effects (font (size 1.27 1.27)) (justify left))
     )
-    (property "Footprint" "" (at 74.422 77.47 90)
+    (property "Footprint" "Resistor_SMD:R_0402_1005Metric" (at 74.422 77.47 90)
       (effects (font (size 1.27 1.27)) hide)
     )
@@
       (effects (font (size 1.27 1.27)) (justify left))
     )
-    (property "Footprint" "" (at 99.822 31.75 90)
+    (property "Footprint" "Resistor_SMD:R_0402_1005Metric" (at 99.822 31.75 90)
       (effects (font (size 1.27 1.27)) hide)
     )
@@
       (effects (font (size 1.27 1.27)) (justify left))
     )
-    (property "Footprint" "" (at 282.9052 227.33 0)
+    (property "Footprint" "Capacitor_SMD:C_0402_1005Metric" (at 282.9052 227.33 0)
       (effects (font (size 1.27 1.27)) hide)
     )
@@
       (effects (font (size 1.27 1.27)) (justify left) hide)
     )
-    (property "Footprint" "" (at 118.872 31.75 90)
+    (property "Footprint" "Resistor_SMD:R_0402_1005Metric" (at 118.872 31.75 90)
       (effects (font (size 1.27 1.27)) hide)
     )
@@
       (effects (font (size 1.27 1.27)) (justify left))
     )
-    (property "Footprint" "" (at 206.7052 227.33 0)
+    (property "Footprint" "Capacitor_SMD:C_0402_1005Metric" (at 206.7052 227.33 0)
       (effects (font (size 1.27 1.27)) hide)
     )
@@
       (effects (font (size 1.27 1.27)))
     )
-    (property "Footprint" "" (at 82.55 113.538 90)
+    (property "Footprint" "Resistor_SMD:R_0402_1005Metric" (at 82.55 113.538 90)
       (effects (font (size 1.27 1.27)) hide)
     )
@@
       (effects (font (size 1.27 1.27)) (justify left))
     )
-    (property "Footprint" "" (at 365.252 119.38 90)
+    (property "Footprint" "Resistor_SMD:R_0402_1005Metric" (at 365.252 119.38 90)
       (effects (font (size 1.27 1.27)) hide)
     )
@@
       (effects (font (size 1.27 1.27)) (justify left))
     )
-    (property "Footprint" "" (at 352.552 119.38 90)
+    (property "Footprint" "Resistor_SMD:R_0402_1005Metric" (at 352.552 119.38 90)
       (effects (font (size 1.27 1.27)) hide)
     )
@@
       (effects (font (size 1.27 1.27)) (justify left))
     )
-    (property "Footprint" "" (at 314.452 119.38 90)
+    (property "Footprint" "Resistor_SMD:R_0402_1005Metric" (at 314.452 119.38 90)
       (effects (font (size 1.27 1.27)) hide)
     )
@@
       (effects (font (size 1.27 1.27)) (justify left))
     )
-    (property "Footprint" "" (at 295.6052 227.33 0)
-      (effects (font (size 1.27 1.27)) hide)
-    )
+    (property "Footprint" "Capacitor_SMD:C_0402_1005Metric" (at 295.6052 227.33 0)
+      (effects (font (size 1.27 1.27)) hide)
+    )
