File: prototype/main.kicad_pcb (KiCad board)
At the start: 2 copper layers, 0 parts

Commit message: tmp
Other:
- board outline added: 90 x 90 mm
Changed lines of the file:
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@@
   )
   (net 0 "")
+  (gr_rect (start 0 -90) (end 90 0)
+    (stroke (width 0.1) (type default)) (fill none) (layer "Edge.Cuts"))
 )
