File: prototype/main.kicad_sch (KiCad schematic)
At the start: 0 parts

Commit message: nrf5240
Other:
- added sheet USB Isolation (usb_iso.kicad_sch)
Changed lines of the file:
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@@
 (kicad_sch (version 20230121) (generator eeschema)
   (paper "A4")
-  (sheet (at 76.2 63.5) (size 25.4 12.7) (fields_autoplaced)
+  (sheet (at 63.5 88.9) (size 25.4 12.7) (fields_autoplaced)
     (stroke (width 0.1524) (type solid))
     (fill (color 0 0 0 0.0000))
-    (property "Sheetname" "PSU" (at 76.2 62.7884 0)
+    (property "Sheetname" "USB Isolation" (at 63.5 88.1884 0)
       (effects (font (size 1.27 1.27)) (justify left bottom))
     )
-    (property "Sheetfile" "psu.kicad_sch" (at 76.2 76.7846 0)
+    (property "Sheetfile" "usb_iso.kicad_sch" (at 63.5 102.1846 0)
       (effects (font (size 1.27 1.27)) (justify left top))
     )
+    (instances
+      (project "main"
+        (path "/71bbf5b6-a913-4747-956a-150714430eae" (page "9"))
+      )
+    )
+  )
+  (sheet (at 114.3 38.1) (size 25.4 12.7) (fields_autoplaced)
+    (stroke (width 0.1524) (type solid))
+    (fill (color 0 0 0 0.0000))
+    (property "Sheetname" "PSU" (at 114.3 37.3884 0)
+      (effects (font (size 1.27 1.27)) (justify left bottom))
+    )
+    (property "Sheetfile" "psu.kicad_sch" (at 114.3 51.3846 0)
+      (effects (font (size 1.27 1.27)) (justify left top))
+    )

Commit message: DAPLink, FT2232H
Other:
- sheet stlink renamed DAP Link
- added sheet RS485 (rs485.kicad_sch)
- sheet BLE ports: added NRF_USB_D_N, NRF_USB_D_P, TRG_CLK, TRG_DIO, TRG_RST, TRG_RXD, TRG_SWO, TRG_TXD; removed none
- sheet Bridge ports: added FT_DTR, FT_RXD, FT_TXD, FT_USB_D_N, FT_USB_D_P; removed none
- sheet DAP Link: file stlink.kicad_sch -> daplink.kicad_sch
- sheet DAP Link ports: added DAP_USB_D_N, DAP_USB_D_P, TRG_CLK, TRG_DIO, TRG_RST, TRG_RXD, TRG_SWO, TRG_TXD; removed none
- sheet Logic ports: added CY_USB_D_N, CY_USB_D_P; removed none
- sheet USB Isolation ports: added HUB_USB_N, HUB_USB_P; removed none
- sheet USB hub ports: added CY_USB_D_N, CY_USB_D_P, DAP_USB_D_N, DAP_USB_D_P, FT_USB_D_N, FT_USB_D_P, HUB_USB_N, HUB_USB_P, NRF_USB_D_N, NRF_USB_D_P; removed none
- note added: "???"
- note added: "C116170"
- note added: "MF-PSMF050X-2"
- note added: "PMCPB5530X"

Commit message: tmp
Other:
- removed sheet USB Isolation
- sheet BLE ports: added BB_ADJ, EXT_PWR_CTRL, LDO_ADJ, NRF_PD_INT, NRF_SCL, NRF_SDA, PWR_EN, PWR_STAT; removed none
- sheet Logic ports: added 3V3_LOGIC; removed none
- sheet PSU ports: added 3V3D_HUB, BB_ADJ, EXT_PWR_CTRL, HUB_USB_N, HUB_USB_P, LDO_ADJ, NRF_PD_INT, NRF_SCL, NRF_SDA, PWR_EN, PWR_STAT; removed none
- sheet RS485 ports: added 3V3D_HUB, RS_LED_R, RS_LED_T; removed none
- note removed: "???"
- note removed: "C116170"
- note removed: "MF-PSMF050X-2"

Commit message: tmp
Parts:
- added U32: STM32G474RCTx, Package_QFP:LQFP-64_10x10mm_P0.5mm, symbol MCU_ST_STM32G4:STM32G474RCTx
Connections:
- new net: U32.15 (VSS), U32.31 (VSS), U32.47 (VSS), U32.63 (VSS)
Other:
- added sheet Electronic Load (eload.kicad_sch)
- sheet uCurrent ports: added DAC; removed none
- note added: "C529413"
- note added: "C529414"
- note added: "STM32G474RBT6"
- note added: "STM32G474RCT6"
- note added: "USB PD controller Controllable PSU 1s/6s charher Discharger/Battery Tester"
Changed lines of the file:
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@@
+    (stroke (width 0) (type default))
+  )
+  (wire (pts (xy 213.36 139.7) (xy 213.36 152.4))
     (stroke (width 0) (type default))
   )
@@
   (wire (pts (xy 152.4 96.52) (xy 149.86 96.52))
     (stroke (width 0) (type default))
+  )
+  (text "C529413" (at 83.82 123.19 0)
+    (effects (font (size 1.27 1.27)) (justify left bottom))
+  )
+  (text "USB PD controller\nControllable PSU\n1s/6s charher\nDischarger/Battery Tester"
+    (at -34.29 107.95 0)
+    (effects (font (size 1.27 1.27)) (justify left bottom))
   )
   (text "PMCPB5530X" (at 5.08 208.28 0)
     (effects (font (size 1.27 1.27)) (justify left bottom))
   )
+  (text "STM32G474RCT6" (at 50.8 125.73 0)
+    (effects (font (size 1.27 1.27)) (justify left bottom))
+  )
+  (text "STM32G474RBT6" (at 83.82 125.73 0)
+    (effects (font (size 1.27 1.27)) (justify left bottom))
+  )
+  (text "C529414" (at 50.8 123.19 0)
+    (effects (font (size 1.27 1.27)) (justify left bottom))
+  )
+  (symbol (lib_id "MCU_ST_STM32G4:STM32G474RCTx") (at -58.42 132.08 0) (unit 1)
+    (in_bom yes) (on_board yes) (dnp no)
+    (property "Reference" "U32" (at -73.66 85.09 0)
+      (effects (font (size 1.27 1.27)) (justify left))
+    )
+    (property "Value" "STM32G474RCTx" (at -54.61 176.53 0)
+      (effects (font (size 1.27 1.27)) (justify left))
+    )
+    (property "Footprint" "Package_QFP:LQFP-64_10x10mm_P0.5mm" (at -73.66 175.26 0)
+      (effects (font (size 1.27 1.27)) (justify right) hide)
+    )
+    (property "Datasheet" "https://www.st.com/resource/en/datasheet/stm32g474rc.pdf" (at -58.42 132.08 0)
+      (effects (font (size 1.27 1.27)) hide)
+    )
+    (pin "1")
+    (pin "10")
+    (pin "11")
+    (pin "12")
+    (pin "13")
+    (pin "14")
+    (pin "15")
+    (pin "16")
+    (pin "17")
+    (pin "18")
+    (pin "19")
+    (pin "2")
+    (pin "20")
+    (pin "21")
+    (pin "22")
+    (pin "23")
+    (pin "24")
+    (pin "25")
+    (pin "26")
+    (pin "27")
+    (pin "28")
+    (pin "29")
+    (pin "3")
+    (pin "30")
+    (pin "31")
+    (pin "32")
+    (pin "33")
+    (pin "34")
+    (pin "35")
+    (pin "36")
+    (pin "37")
+    (pin "38")
+    (pin "39")
+    (pin "4")
+    (pin "40")
+    (pin "41")
+    (pin "42")
+    (pin "43")
+    (pin "44")
+    (pin "45")
+    (pin "46")
+    (pin "47")
+    (pin "48")
+    (pin "49")
+    (pin "5")
+    (pin "50")
+    (pin "51")
+    (pin "52")
+    (pin "53")
+    (pin "54")
+    (pin "55")
+    (pin "56")
+    (pin "57")
+    (pin "58")
+    (pin "59")
+    (pin "6")
+    (pin "60")
+    (pin "61")
+    (pin "62")
+    (pin "63")
+    (pin "64")
+    (pin "7")
+    (pin "8")
+    (pin "9")
+    (instances
+      (project "main"
+        (path "/71bbf5b6-a913-4747-956a-150714430eae"
+          (reference "U32") (unit 1)
+        )
+      )
+    )
+  )
   (sheet (at 76.2 127) (size 25.4 38.1) (fields_autoplaced)
     (stroke (width 0.1524) (type solid))
@@
     )
   )
+  (sheet (at 190.5 152.4) (size 25.4 12.7) (fields_autoplaced)
+    (stroke (width 0.1524) (type solid))
+    (fill (color 0 0 0 0.0000))
+    (property "Sheetname" "Electronic Load" (at 190.5 151.6884 0)
+      (effects (font (size 1.27 1.27)) (justify left bottom))
+    )
+    (property "Sheetfile" "eload.kicad_sch" (at 190.5 165.6846 0)
+      (effects (font (size 1.27 1.27)) (justify left top))
+    )
+    (pin "DAC" input (at 213.36 152.4 90)
+      (effects (font (size 1.27 1.27)) (justify right))
+    )
+    (instances
+      (project "main"
+        (path "/71bbf5b6-a913-4747-956a-150714430eae" (page "10"))
+      )
+    )
+  )
   (sheet (at 152.4 106.68) (size 25.4 33.02) (fields_autoplaced)
     (stroke (width 0.1524) (type solid))
@@
       (effects (font (size 1.27 1.27)) (justify left top))
     )
-    (instances
+    (pin "DAC" input (at 213.36 139.7 270)
+      (effects (font (size 1.27 1.27)) (justify left))
+    )
+    (instances
