File: prototype/psu.kicad_sch (KiCad schematic)
At the start: 0 parts

Commit message: DAPLink, FT2232H
Parts:
- added J13: PCB_EDGE+, symbol Connector:Conn_01x01_Pin
- added J15: PCB_EDGE-, symbol Connector:Conn_01x01_Pin
- added J16: Terminal+, symbol Connector:Conn_01x01_Socket
- added J17: Terminal-, symbol Connector:Conn_01x01_Socket
Connections:
- new net GND: J15.1 (Pin_1), J17.1 (Pin_1)
- new net VDC: J13.1 (Pin_1), J16.1 (Pin_1)
Other:
- note added: "BQ24105RHLR"
- note added: "wide-range: 3.3 ... 24V"
Changed lines of the file:
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@@
 (kicad_sch (version 20230121) (generator eeschema)
   (paper "A4")
+  (junction (at 40.64 38.1) (diameter 0) (color 0 0 0 0)
+  )
+  (junction (at 40.64 33.02) (diameter 0) (color 0 0 0 0)
+  )
+  (wire (pts (xy 40.64 38.1) (xy 40.64 40.64))
+    (stroke (width 0) (type default))
+  )
+  (wire (pts (xy 38.1 38.1) (xy 40.64 38.1))
+    (stroke (width 0) (type default))
+  )
+  (wire (pts (xy 40.64 30.48) (xy 40.64 33.02))
+    (stroke (width 0) (type default))
+  )
+  (wire (pts (xy 52.07 33.02) (xy 52.07 30.48))
+    (stroke (width 0) (type default))
+  )
+  (wire (pts (xy 40.64 38.1) (xy 52.07 38.1))
+    (stroke (width 0) (type default))
+  )
+  (wire (pts (xy 52.07 38.1) (xy 52.07 40.64))
+    (stroke (width 0) (type default))
+  )
+  (wire (pts (xy 38.1 33.02) (xy 40.64 33.02))
+    (stroke (width 0) (type default))
+  )
+  (wire (pts (xy 40.64 33.02) (xy 52.07 33.02))
+    (stroke (width 0) (type default))
+  )
+  (text "wide-range: 3.3 ... 24V" (at 38.1 36.83 0)
+    (effects (font (size 1.27 1.27)) (justify left bottom))
+  )
+  (text "BQ24105RHLR" (at 74.93 34.29 0)
+    (effects (font (size 1.27 1.27)) (justify left bottom))
+  )
+  (symbol (lib_id "Connector:Conn_01x01_Pin") (at 33.02 38.1 0) (unit 1)
+    (in_bom no) (on_board yes) (dnp no)
+    (property "Reference" "J15" (at 33.02 36.83 0)
+      (effects (font (size 1.27 1.27)))
+    )
+    (property "Value" "PCB_EDGE-" (at 26.67 38.1 0)
+      (effects (font (size 1.27 1.27)))
+    )
+    (property "Footprint" "" (at 33.02 38.1 0)
+      (effects (font (size 1.27 1.27)) hide)
+    )
+    (property "Datasheet" "~" (at 33.02 38.1 0)
+      (effects (font (size 1.27 1.27)) hide)
+    )
+    (pin "1")
+    (instances
+      (project "main"
+        (path "/71bbf5b6-a913-4747-956a-150714430eae/10961a25-19b6-4f34-b84e-851f54b2404d"
+          (reference "J15") (unit 1)
+        )
+      )
+    )
+  )
+  (symbol (lib_id "power:GND") (at 52.07 40.64 0) (unit 1)
+    (in_bom yes) (on_board yes) (dnp no) (fields_autoplaced)
+    (property "Reference" "#PWR073" (at 52.07 46.99 0)
+      (effects (font (size 1.27 1.27)) hide)
+    )
+    (property "Value" "GND" (at 52.07 45.72 0)
+      (effects (font (size 1.27 1.27)))
+    )
+    (property "Footprint" "" (at 52.07 40.64 0)
+      (effects (font (size 1.27 1.27)) hide)
+    )
+    (property "Datasheet" "" (at 52.07 40.64 0)
+      (effects (font (size 1.27 1.27)) hide)
+    )
+    (pin "1")
+    (instances
+      (project "main"
+        (path "/71bbf5b6-a913-4747-956a-150714430eae/10961a25-19b6-4f34-b84e-851f54b2404d"
+          (reference "#PWR073") (unit 1)
+        )
+      )
+    )
+  )
+  (symbol (lib_id "Connector:Conn_01x01_Pin") (at 33.02 33.02 0) (unit 1)
+    (in_bom no) (on_board yes) (dnp no)
+    (property "Reference" "J13" (at 33.02 31.75 0)
+      (effects (font (size 1.27 1.27)))
+    )
+    (property "Value" "PCB_EDGE+" (at 26.67 33.02 0)
+      (effects (font (size 1.27 1.27)))
+    )
+    (property "Footprint" "" (at 33.02 33.02 0)
+      (effects (font (size 1.27 1.27)) hide)
+    )
+    (property "Datasheet" "~" (at 33.02 33.02 0)
+      (effects (font (size 1.27 1.27)) hide)
+    )
+    (pin "1")
+    (instances
+      (project "main"
+        (path "/71bbf5b6-a913-4747-956a-150714430eae/10961a25-19b6-4f34-b84e-851f54b2404d"
+          (reference "J13") (unit 1)
+        )
+      )
+    )
+  )
+  (symbol (lib_id "Connector:Conn_01x01_Socket") (at 40.64 25.4 90) (unit 1)
+    (in_bom yes) (on_board yes) (dnp no)
+    (property "Reference" "J16" (at 41.91 26.67 90)
+      (effects (font (size 1.27 1.27)) (justify right))
+    )
+    (property "Value" "Terminal+" (at 40.64 24.13 90)
+      (effects (font (size 1.27 1.27)))
+    )
+    (property "Footprint" "" (at 40.64 25.4 0)
+      (effects (font (size 1.27 1.27)) hide)
+    )
+    (property "Datasheet" "~" (at 40.64 25.4 0)
+      (effects (font (size 1.27 1.27)) hide)
+    )
+    (pin "1")
+    (instances
+      (project "main"
+        (path "/71bbf5b6-a913-4747-956a-150714430eae/10961a25-19b6-4f34-b84e-851f54b2404d"
+          (reference "J16") (unit 1)
+        )
+      )
+    )
+  )
+  (symbol (lib_id "power:VDC") (at 52.07 30.48 0) (unit 1)
+    (in_bom yes) (on_board yes) (dnp no)
+    (property "Reference" "#PWR074" (at 52.07 33.02 0)
+      (effects (font (size 1.27 1.27)) hide)
+    )
+    (property "Value" "VDC" (at 52.07 26.67 0)
+      (effects (font (size 1.27 1.27)))
+    )
+    (property "Footprint" "" (at 52.07 30.48 0)
+      (effects (font (size 1.27 1.27)) hide)
+    )
+    (property "Datasheet" "" (at 52.07 30.48 0)
+      (effects (font (size 1.27 1.27)) hide)
+    )
+    (pin "1")
+    (instances
+      (project "main"
+        (path "/71bbf5b6-a913-4747-956a-150714430eae/10961a25-19b6-4f34-b84e-851f54b2404d"
+          (reference "#PWR074") (unit 1)
+        )
+      )
+    )
+  )
+  (symbol (lib_id "Connector:Conn_01x01_Socket") (at 40.64 45.72 270) (unit 1)
+    (in_bom yes) (on_board yes) (dnp no)
+    (property "Reference" "J17" (at 41.91 44.45 90)
+      (effects (font (size 1.27 1.27)) (justify left))
+    )
+    (property "Value" "Terminal-" (at 40.64 46.99 90)
+      (effects (font (size 1.27 1.27)))
+    )
+    (property "Footprint" "" (at 40.64 45.72 0)
+      (effects (font (size 1.27 1.27)) hide)
+    )
+    (property "Datasheet" "~" (at 40.64 45.72 0)
+      (effects (font (size 1.27 1.27)) hide)
+    )
+    (pin "1")
+    (instances
+      (project "main"
+        (path "/71bbf5b6-a913-4747-956a-150714430eae/10961a25-19b6-4f34-b84e-851f54b2404d"
+          (reference "J17") (unit 1)
+        )
+      )
+    )
+  )
 )

Commit message: tmp
Parts:
- removed J16: Terminal+, symbol Connector:Conn_01x01_Socket
- removed J17: Terminal-, symbol Connector:Conn_01x01_Socket
- added BT1: LP605590, symbol Device:Battery_Cell
- added C104: C, symbol Device:C
- added C105, C106, C107, C110, C131, C83, C87, C88, C89: 0.1u, symbol Device:C
- added C108, C109: 330p, symbol Device:C
- added C111, C112, C132, C133, C134, C135, C136, C137: ??, symbol Device:C
- added C113, C114: 47n, symbol Device:C
- added C115, C118: 150p, symbol Device:C
- added C116: 1n, symbol Device:C
- added C117: 10n, symbol Device:C
- added C119, C120, C121, C122, C123, C124, C126, C127, C129, C80, C82, C84, C85, C86: 10u, symbol Device:C
- added C125, C128: 47u, symbol Device:C
- added C130: 1u, symbol Device:C
- added D13: D_Zener, symbol Device:D_Zener
- added D14, D20, D21, D22, D23, D25, D27, D33, D35, D37: SMA4007, Diode_SMD:D_SMA, symbol Device:D
- added D24: B5819W, Diode_SMD:D_SOD-123, symbol Device:D_Zener
- added D26, D32: D_Schottky, symbol Device:D_Schottky
- added D28, D29, D30, D31: 12V, symbol Device:D_Zener
- added D34: D_Schottky_Small, symbol Device:D_Schottky_Small
- added F1, F2, F3, F4: 12T.30000063AG12S1B02, Fuse:Fuse_1206_3216Metric, symbol Device:Fuse
- added J16, J26, J27: +, symbol Connector:Screw_Terminal_01x01
- added J17, J25, J28: -, symbol Connector:Screw_Terminal_01x01
- added J19: Battery, symbol Connector_Generic:Conn_01x02
- added J29: PCB_EDGE-, symbol Connector:Conn_01x01_Pin
- added J30: PCB_EDGE+, symbol Connector:Conn_01x01_Pin
- added J7: TYPE-C-31-M-12, MAS_Package_std:USB_C_Receptacle_HRO_TYPE-C-31-M-12, symbol Connector:USB_C_Receptacle_USB2.0
- added L10, L11, L14, L15, L16: L, symbol Device:L
- added L12: 2.2u, Inductor_SMD:L_Wuerth_WE-PD2-Typ-XL, symbol Device:L
- added L13: 1u, symbol Device:L
- added L9: 1.5u, symbol Device:L
- added Q10, Q6, Q9: CSD17551Q3A, Package_TO_SOT_SMD:TDSON-8-1, symbol Transistor_FET:CSD17551Q5A
- added Q12, Q16, Q17, Q21, Q22, Q23, Q27, Q28: 2N7002, Package_TO_SOT_SMD:SOT-23, symbol Transistor_FET:2N7002
- added Q13, Q14, Q18: ECH8690, Package_TO_SOT_SMD:OnSemi_ECH8, symbol chrns_transistor:ECH8690
- added Q15, Q19, Q20: PNP, symbol Simulation_SPICE:PNP
- added Q7: DMP3035SFG-7, Package_SON:Diodes_PowerDI3333-8, symbol Transistor_FET:DMP3013SFV
- added Q8: 2N7002ET1G-ES, Package_TO_SOT_SMD:SOT-23, symbol Transistor_FET:2N7002E
- added R101, R95, R97, R98: 330k, symbol Device:R
- added R105, R106: 7.5k, symbol Device:R
- added R107: 0.1, symbol Device:R
- added R108, R112, R113, R114, R116, R118, R120, R123, R125, R126, R127, R128, R129, R132, R133: 10k, symbol Device:R
- added R111, R115, R117, R119, R121, R122, R124: 100k, symbol Device:R
- added R76, R77: R, symbol Device:R
- added R96, R99: 33k, symbol Device:R
- added SW9: !K2-1102AQ-N4CW-01, Button_Switch_THT:SW_Tactile_SPST_Angled_PTS645Vx83-2LFS, symbol Switch:SW_Push
- added TH1: Thermistor_NTC, symbol Device:Thermistor_NTC
- added U11: ADP2504ACPZ-R7, Package_DFN_QFN:DFN-10-1EP_3x3mm_P0.5mm_EP1.65x2.38mm, symbol chrns_ic_power:ADP2504
- added U12: ADP1708, Package_DFN_QFN:DFN-8-1EP_3x3mm_P0.5mm_EP1.65x2.38mm, symbol chrns_ic_power:ADP1708
- added U22: BQ24105RHLR, Package_DFN_QFN:Texas_VQFN-RHL-20, symbol chrns_ic_power:BQ24105
- added U23: FUSB302BMPX, Package_DFN_QFN:WQFN-14-1EP_2.5x2.5mm_P0.5mm_EP1.45x1.45mm, symbol Interface_USB:FUSB302BMPX
- added U25: BQ25703A, Package_DFN_QFN:WQFN-32-1EP_5x5mm_P0.5mm_EP3.1x3.1mm, symbol chrns_ic_power:BQ25703A
- added U28: SiP32431DR3, Package_TO_SOT_SMD:SOT-363_SC-70-6, symbol Power_Management:SiP32431DR3
- added U9: BQ25611D, Package_DFN_QFN:Texas_S-PWQFN-N24_EP2.7x2.7mm, symbol chrns_ic_power:BQ25611D
Connections:
- net GND: now also C105.2, C106.2, C107.2, C108.2, C109.2, C110.2, C111.2, C112.2, C115.2, C116.2, C117.2, C118.1, C119.2, C120.2, C121.2, C122.2, C123.2, C124.2, C126.2, C127.2, C128.2, C129.2, C130.2, C132.2, C133.2, C134.2, C135.2, C136.2, C137.2, C80.2, C82.2, C83.2, C84.2, C85.2, C86.2, C87.2, C88.2, C89.2, D22.2 (A), D23.2 (A), D27.2 (A), D32.2 (A), D37.2 (A), J7.A1 (GND), J7.A12 (GND), J7.B1 (GND), J7.B12 (GND), J7.S1 (SHIELD), Q12.2 (S), Q13.1, Q14.5, Q14.6, Q16.2 (S), Q22.2 (S), Q23.2 (S), Q27.2 (S), Q6.1 (S), Q6.2 (S), Q6.3 (S), Q7.1 (S), Q7.2 (S), Q7.3 (S), R105.2, R106.2, R111.1, R117.2, R119.2, R121.2, R124.2, R129.2, R77.2, R96.2, R99.2, TH1.2, U11.11 (PAD), U11.3 (PGND), U11.9 (AGND), U12.2 (GND), U12.9 (PAD), U22.10 (VSS), U22.17 (PGND), U22.18 (PGND), U22.21 (PAD), U23.15 (GND), U23.8 (GND), U23.9 (GND), U25.27 (PGND), U25.33 (PAD), U28.2 (GND), U28.5 (GND), U9.17 (GND), U9.18 (GND), U9.25 (PAD), U9.9 (~{CE}); no longer J15.1 (Pin_1)
- net VDC: now also C86.1, R98.1, U12.5 (OUT), U12.6 (OUT), U12.7 (SENSE); no longer J13.1 (Pin_1)
- new net: Q16.3 (D), R116.1
- new net: D28.2 (A), Q14.2, R115.1, R116.2
- new net: R101.1, R98.2, R99.1, U12.8 (ADJ)
- new net: R95.2, R96.1, R97.1
- new net: C126.1, L13.2, U9.15 (SYS), U9.16 (SYS)
- new net: Q16.1 (G), R118.2, R119.1
- new net: C113.1, L12.1, Q6.5 (D), Q9.1 (S), Q9.2 (S), Q9.3 (S), U25.32 (SW1)
- new net: C113.2, U25.30 (BTST1)
- new net: D14.1 (K), D25.2 (A), Q22.3 (D)
- new net: C114.1, L12.2, Q10.1 (S), Q10.2 (S), Q10.3 (S), Q7.5 (D), U25.23 (SW2)
- new net: C114.2, U25.25 (BTST2)
- new net: Q20.1 (C), Q21.1 (G), R129.1
- new net: D25.1 (K), F2.1, Q17.3 (D), Q19.3 (E), R127.2
- new net: C132.1, F2.2, L14.1
- new net: D26.2 (A), D34.1 (K), J17.1 (Pin_1), Q27.3 (D)
- new net: R108.2, U23.5 (INT_N)
- new net: Q12.1 (G), R120.2, R121.1
- new net: C116.1, C117.1, Q9.5 (D)
- new net: D32.1 (K), J26.1 (Pin_1), Q28.2 (S), R133.1
- new net: Q15.1 (C), Q28.1 (G), R133.2
- new net: R105.1, U22.9 (ISET2)
- new net: C119.1, C120.1, C121.1, C122.1, C123.1, C124.1, Q10.5 (D)
- new net: D27.1 (K), Q17.2 (S), R126.1
- new net: C134.1, F3.2, L15.1
- new net: C111.1, F1.2, L11.1
- new net: Q10.4 (G), U25.24 (HIDRV2)
- new net: C118.2, Q7.4 (G), U25.26 (LODRV2)
- new net: C115.1, Q6.4 (G), U25.29 (LODRV1)
- new net: Q9.4 (G), U25.31 (HIDRV1)
- new net: D21.1 (K), D23.1 (K), F1.1
- new net: D29.2 (A), Q14.4, R114.1, R117.1
- new net: D26.1 (K), D34.2 (A), F4.1, Q15.3 (E), Q28.3 (D), R132.2
- new net: R106.1, U22.8 (ISET1)
- new net: C136.1, F4.2, L16.1
- new net: L9.1, U11.4 (SW1)
- new net: L9.2, U11.2 (SW2)
- new net: D31.2 (A), Q13.2, R124.1, R125.1
- new net: D24.2 (A), R111.2, R112.1, SW9.2
- new net: C125.1, L13.1, U9.19 (SW), U9.20 (SW)
- new net: Q17.1 (G), Q19.1 (C), R126.2
- new net: C131.1, D24.1 (K), R113.2, U28.3 (ON)
- new net: Q12.3 (D), R123.1
- new net: D30.2 (A), Q13.4, Q18.4, R122.1, R123.2
- new net: Q15.2 (B), R132.1
- new net: D35.2 (A), Q20.2 (B), R128.1
- new net: C128.1, U9.22 (REGN)
- new net: D14.2 (A), Q19.2 (B), R127.1
- new net: C125.2, U9.21 (BTST)
- new net: D30.1 (K), Q13.3, Q18.3
- new net: Q18.7, Q18.8
- new net +BATT: C127.1, J19.1 (Pin_1), R76.1, SW9.1, U28.4 (IN), U9.10 (BATSNS), U9.13 (BAT), U9.14 (BAT)
- new net -BATT: J19.2 (Pin_2)
- new net BB_ADJ: R97.2
- new net BQ_QON: U9.12 (~{QON})
- new net BQ_TS: R76.2, R77.1, TH1.1, U9.11 (TS)
- new net CHARGE: U22.2 (STAT1)
- new net DONE: U22.19 (STAT2)
- new net EXT_PWR_CTRL: Q27.1 (G)
- new net HUB_USB_N: J7.A7 (D-), J7.B7 (D-), U9.3 (D-)
- new net HUB_USB_P: J7.A6 (D+), J7.B6 (D+), U9.2 (D+)
- new net IN: U22.3 (IN), U22.4 (IN), U22.6 (VCC)
- new net LDO_ADJ: R101.2
- new net NRF_SCL: U23.6 (SCL), U25.13 (SCL), U9.6 (SDA)
- new net NRF_SDA: U23.7 (SDA), U25.12 (SDA), U9.5 (SCL)
- new net OUT: U22.1 (OUT), U22.20 (OUT)
- new net PD_CC1: C109.1, J7.A5 (CC1), U23.10 (CC1), U23.11 (CC1)
- new net PD_CC2: C108.1, J7.B5 (CC2), U23.1 (CC2), U23.14 (CC2)
- new net PMID: C129.1, U9.23 (PMID)
- new net PRESENT: U22.5 (~{PG})
- new net PSU_EN: U11.6 (EN), U12.1 (EN)
- new net PWR+: D20.1 (K), D21.2 (A), D28.1 (K), D33.1 (K), D37.1 (K), F3.1, J13.1 (Pin_1), J16.1 (Pin_1), J27.1 (Pin_1), J30.1 (Pin_1), Q14.1, Q18.5, Q18.6, Q20.3 (E), Q21.2 (S), Q21.3 (D), R114.2, R125.2, R128.2
- new net PWR-: D20.2 (A), D22.1 (K), D29.1 (K), D31.1 (K), D33.2 (A), D35.1 (K), J15.1 (Pin_1), J25.1 (Pin_1), J28.1 (Pin_1), J29.1 (Pin_1), Q13.7, Q13.8, Q14.3, Q23.3 (D)
- new net PWR_EN: C131.2, R113.1
- new net PWR_STAT: R112.2
- new net TTC: C89.1
- new net VBUS: C110.1, C112.1, C130.1, C133.1, C135.1, C137.1, J7.A4 (VBUS), J7.A9 (VBUS), J7.B4 (VBUS), J7.B9 (VBUS), L11.2, L14.2, L15.2, L16.2, Q13.5, Q13.6, Q14.7, Q14.8, R115.2, R122.2, U23.2 (VBUS), U9.1 (VAC), U9.24 (VBUS)
- new net VDD: C105.1, C106.1, C107.1, C80.1, C83.1, R108.1, U11.5 (PVIN), U11.8 (VIN), U23.12 (VCONN), U23.13 (VCONN), U23.3 (VDD), U23.4 (VDD), U28.1 (OUT)
- new net VDD_PRE: C82.1, C84.1, C85.1, R95.1, U11.1 (VOUT), U12.3 (IN), U12.4 (IN)
- new net VTSB: C88.1
- no-connect marks 0 -> 4
Other:
- note added: "2N7002ET1G"
- note added: "3.3 ... 20V"
- note added: "5V ... 20V"
- note added: "???"
- note added: "Battery"
- note added: "C2861620"
- note added: "CSD17551Q3A"
- note added: "CSD23382F4"
- note added: "DMP3035SFG-7"
- note added: "ERR"
- note added: "External power supply"
- note added: "IHLP3232CZER2R2M01"
- note added: "TPS2561DRCR"
- note added: "USB Power Delivery"
- note added: "to uCurrent"
- note removed: "BQ24105RHLR"
- note removed: "wide-range: 3.3 ... 24V"
- moved on the sheet: J13, J15

Commit message: tmp
Parts:
- removed C111, C112, C132, C133, C134, C135: ??, symbol Device:C
- removed D14, D20, D21, D22, D23, D25, D27, D33, D35, D37: SMA4007, Diode_SMD:D_SMA, symbol Device:D
- removed D28, D29: 12V, symbol Device:D_Zener
- removed F1, F2, F3: 12T.30000063AG12S1B02, Fuse:Fuse_1206_3216Metric, symbol Device:Fuse
- removed J13, J30: PCB_EDGE+, symbol Connector:Conn_01x01_Pin
- removed J15, J29: PCB_EDGE-, symbol Connector:Conn_01x01_Pin
- removed J25: -, symbol Connector:Screw_Terminal_01x01
- removed L11, L14, L15: L, symbol Device:L
- removed Q14, Q18: ECH8690, Package_TO_SOT_SMD:OnSemi_ECH8, symbol chrns_transistor:ECH8690
- removed Q16, Q17, Q21, Q22: 2N7002, Package_TO_SOT_SMD:SOT-23, symbol Transistor_FET:2N7002
- removed Q19, Q20: PNP, symbol Simulation_SPICE:PNP
- removed R114, R116, R118, R126, R127, R128, R129: 10k, symbol Device:R
- removed R115, R117, R119: 100k, symbol Device:R
- added D23: 12V, symbol Device:D_Zener
- added D39, D40: D_Schottky, symbol Device:D_Schottky
- added J15: +, symbol Connector:Screw_Terminal_01x01
- added Q11, Q42, Q43: ECH8690, Package_TO_SOT_SMD:OnSemi_ECH8, symbol chrns_transistor:ECH8690
- added R212, R215: 10k, Resistor_SMD:R_0402_1005Metric, symbol Device:R
- added R213, R214: 100k, Resistor_SMD:R_0402_1005Metric, symbol Device:R
- C104, C105, C106, C107, C108, C109, C110, C113, C114, C115, C116, C117, C118, C119, C120, C121, C122, C123, C124, C125, C126, C127, C128, C129, C130, C131, C80, C82, C83, C84, C85, C86, C87, C88, C89: footprint (none) -> Capacitor_SMD:C_0402_1005Metric
- J16: value + -> -
- R101, R105, R106, R107, R108, R111, R112, R113, R120, R121, R122, R123, R124, R125, R132, R133, R76, R77, R95, R96, R97, R98, R99: footprint (none) -> Resistor_SMD:R_0402_1005Metric
Connections:
- net GND: now also J16.1 (Pin_1), J28.1 (Pin_1), Q13.7, Q13.8, D39.2 (A), Q11.7, Q11.8, R213.2; no longer Q13.1
- net PWR+: now also Q13.5, Q13.6, J15.1 (Pin_1), Q43.5, Q43.6; no longer J16.1 (Pin_1)
- net VBUS: now also C116.1, C117.1, Q9.5 (D), Q11.5, Q11.6, Q42.5, Q42.6, R214.2; no longer Q13.5, Q13.6
- net at D26.2 (A), D34.1 (K), J17.1 (Pin_1)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: now also D39.1 (K)
- net NRF_PD_INT: now reaches R108.2, U23.5 (INT_N)
- net at D32.1 (K), J26.1 (Pin_1), Q28.2 (S)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: now also D40.2 (A)
- net at D26.1 (K), F4.1, Q15.3 (E)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: now also D40.1 (K); no longer D34.2 (A)
- net at D31.2 (A), Q13.2, R124.1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: now also Q11.2
- net at D30.2 (A), Q13.4, R122.1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: now also Q11.4
- net at Q15.2 (B), R132.1: now also D34.2 (A)
- net at Q23.1 (G): now also R212.2, R213.1
- net at D30.1 (K), Q13.3: now also Q11.3
- removed net PWR-: D31.1 (K), J28.1 (Pin_1), Q13.7, Q13.8, Q23.3 (D)
- new net: D31.1 (K), Q11.1, Q13.1
- new net: Q23.3 (D), R215.1
- new net: D23.2 (A), Q42.4, Q43.4, R214.1, R215.2
- new net: D23.1 (K), Q42.3, Q43.3
Other:
- note added: "C341531"
- note added: "DLW5BTM142TQ2"
- note removed: "3.3 ... 20V"
- note removed: "ERR"
- moved on the sheet: C113, C114, C115, C116, C117, C118, C119, C120, C121, C122, C123, C124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
