File: prototype/uCurrent.kicad_sch (KiCad schematic)
At the start: 0 parts

Commit message: nrf5240
Parts:
- added C2: 0.1u, Capacitor_SMD:C_0402_1005Metric, symbol Device:C
- added R56: 0.3, Resistor_SMD:R_2512_6332Metric, symbol Device:R
- added U8: INA219AxDCN, Package_TO_SOT_SMD:SOT-23-8, symbol Sensor_Energy:INA219AxDCN
Connections:
- new net GND: C2.2, U8.3 (GND), U8.7 (A0), U8.8 (A1)
- new net SCL: U8.5 (SCL)
- new net SDA: U8.6 (SDA)
- new net VIN: R56.1, U8.1 (IN+)
- new net VOUT: R56.2, U8.2 (IN-)
Other:
- note added: "mAmp-meter"
Changed lines of the file:
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@@
 (kicad_sch (version 20230121) (generator eeschema)
   (paper "A4")
+  (junction (at 76.2 81.28) (diameter 0) (color 0 0 0 0)
+  )
+  (junction (at 63.5 87.63) (diameter 0) (color 0 0 0 0)
+  )
+  (junction (at 44.45 82.55) (diameter 0) (color 0 0 0 0)
+  )
+  (junction (at 44.45 69.85) (diameter 0) (color 0 0 0 0)
+  )
+  (wire (pts (xy 44.45 82.55) (xy 44.45 80.01))
+    (stroke (width 0) (type default))
+  )
+  (wire (pts (xy 50.8 69.85) (xy 44.45 69.85))
+    (stroke (width 0) (type default))
+  )
+  (wire (pts (xy 76.2 81.28) (xy 76.2 87.63))
+    (stroke (width 0) (type default))
+  )
+  (wire (pts (xy 63.5 87.63) (xy 63.5 88.9))
+    (stroke (width 0) (type default))
+  )
+  (wire (pts (xy 63.5 86.36) (xy 63.5 87.63))
+    (stroke (width 0) (type default))
+  )
+  (wire (pts (xy 44.45 63.5) (xy 44.45 69.85))
+    (stroke (width 0) (type default))
+  )
+  (wire (pts (xy 50.8 78.74) (xy 50.8 82.55))
+    (stroke (width 0) (type default))
+  )
+  (wire (pts (xy 73.66 78.74) (xy 76.2 78.74))
+    (stroke (width 0) (type default))
+  )
+  (wire (pts (xy 76.2 78.74) (xy 76.2 81.28))
+    (stroke (width 0) (type default))
+  )
+  (wire (pts (xy 63.5 63.5) (xy 63.5 66.04))
+    (stroke (width 0) (type default))
+  )
+  (wire (pts (xy 53.34 78.74) (xy 50.8 78.74))
+    (stroke (width 0) (type default))
+  )
+  (wire (pts (xy 73.66 71.12) (xy 88.9 71.12))
+    (stroke (width 0) (type default))
+  )
+  (wire (pts (xy 73.66 73.66) (xy 88.9 73.66))
+    (stroke (width 0) (type default))
+  )
+  (wire (pts (xy 44.45 82.55) (xy 44.45 88.9))
+    (stroke (width 0) (type default))
+  )
+  (wire (pts (xy 73.66 81.28) (xy 76.2 81.28))
+    (stroke (width 0) (type default))
+  )
+  (wire (pts (xy 63.5 87.63) (xy 76.2 87.63))
+    (stroke (width 0) (type default))
+  )
+  (wire (pts (xy 50.8 82.55) (xy 44.45 82.55))
+    (stroke (width 0) (type default))
+  )
+  (wire (pts (xy 101.6 69.85) (xy 101.6 72.39))
+    (stroke (width 0) (type default))
+  )
+  (wire (pts (xy 44.45 69.85) (xy 44.45 72.39))
+    (stroke (width 0) (type default))
+  )
+  (wire (pts (xy 53.34 73.66) (xy 50.8 73.66))
+    (stroke (width 0) (type default))
+  )
+  (wire (pts (xy 101.6 80.01) (xy 101.6 82.55))
+    (stroke (width 0) (type default))
+  )
+  (wire (pts (xy 50.8 73.66) (xy 50.8 69.85))
+    (stroke (width 0) (type default))
+  )
+  (text "mAmp-meter" (at 69.85 91.44 0)
+    (effects (font (size 1.27 1.27)) (justify left bottom))
+  )
+  (label "SCL" (at 88.9 73.66 180) (fields_autoplaced)
+    (effects (font (size 1.27 1.27)) (justify right bottom))
+  )
+  (label "SDA" (at 88.9 71.12 180) (fields_autoplaced)
+    (effects (font (size 1.27 1.27)) (justify right bottom))
+  )
+  (label "VIN" (at 44.45 63.5 0) (fields_autoplaced)
+    (effects (font (size 1.27 1.27)) (justify left bottom))
+  )
+  (label "VOUT" (at 44.45 88.9 0) (fields_autoplaced)
+    (effects (font (size 1.27 1.27)) (justify left bottom))
+  )
+  (symbol (lib_id "power:GND") (at 63.5 88.9 0) (unit 1)
+    (in_bom yes) (on_board yes) (dnp no)
+    (property "Reference" "#PWR017" (at 63.5 95.25 0)
+      (effects (font (size 1.27 1.27)) hide)
+    )
+    (property "Value" "GND" (at 63.5 92.71 0)
+      (effects (font (size 1.27 1.27)))
+    )
+    (property "Footprint" "" (at 63.5 88.9 0)
+      (effects (font (size 1.27 1.27)) hide)
+    )
+    (property "Datasheet" "" (at 63.5 88.9 0)
+      (effects (font (size 1.27 1.27)) hide)
+    )
+    (pin "1")
+    (instances
+      (project "main"
+        (path "/71bbf5b6-a913-4747-956a-150714430eae/8c222416-b30d-49c6-bdd9-9c9a8764b515"
+          (reference "#PWR017") (unit 1)
+        )
+        (path "/71bbf5b6-a913-4747-956a-150714430eae/ca3bda99-bde3-405c-8940-a13088a856d3"
+          (reference "#PWR044") (unit 1)
+        )
+      )
+    )
+  )
+  (symbol (lib_id "Sensor_Energy:INA219AxDCN") (at 63.5 76.2 0) (unit 1)
+    (in_bom yes) (on_board yes) (dnp no)
+    (property "Reference" "U8" (at 55.88 67.31 0)
+      (effects (font (size 1.27 1.27)) (justify left))
+    )
+    (property "Value" "INA219AxDCN" (at 64.77 67.31 0)
+      (effects (font (size 1.27 1.27)) (justify left))
+    )
+    (property "Footprint" "Package_TO_SOT_SMD:SOT-23-8" (at 80.01 85.09 0)
+      (effects (font (size 1.27 1.27)) hide)
+    )
+    (property "Datasheet" "http://www.ti.com/lit/ds/symlink/ina219.pdf" (at 72.39 78.74 0)
+      (effects (font (size 1.27 1.27)) hide)
+    )
+    (pin "1")
+    (pin "2")
+    (pin "3")
+    (pin "4")
+    (pin "5")
+    (pin "6")
+    (pin "7")
+    (pin "8")
+    (instances
+      (project "main"
+        (path "/71bbf5b6-a913-4747-956a-150714430eae/ca3bda99-bde3-405c-8940-a13088a856d3"
+          (reference "U8") (unit 1)
+        )
+      )
+    )
+  )
+  (symbol (lib_id "power:GND") (at 101.6 82.55 0) (unit 1)
+    (in_bom yes) (on_board yes) (dnp no)
+    (property "Reference" "#PWR017" (at 101.6 88.9 0)
+      (effects (font (size 1.27 1.27)) hide)
+    )
+    (property "Value" "GND" (at 101.6 86.36 0)
+      (effects (font (size 1.27 1.27)))
+    )
+    (property "Footprint" "" (at 101.6 82.55 0)
+      (effects (font (size 1.27 1.27)) hide)
+    )
+    (property "Datasheet" "" (at 101.6 82.55 0)
+      (effects (font (size 1.27 1.27)) hide)
+    )
+    (pin "1")
+    (instances
+      (project "main"
+        (path "/71bbf5b6-a913-4747-956a-150714430eae/8c222416-b30d-49c6-bdd9-9c9a8764b515"
+          (reference "#PWR017") (unit 1)
+        )
+        (path "/71bbf5b6-a913-4747-956a-150714430eae/ca3bda99-bde3-405c-8940-a13088a856d3"
+          (reference "#PWR045") (unit 1)
+        )
+      )
+    )
+  )
+  (symbol (lib_id "Device:C") (at 101.6 76.2 0) (unit 1)
+    (in_bom yes) (on_board yes) (dnp no)
+    (property "Reference" "C2" (at 105.41 73.66 0)
+      (effects (font (size 1.27 1.27)) (justify left))
+    )
+    (property "Value" "0.1u" (at 105.41 76.2 0)
+      (effects (font (size 1.27 1.27)) (justify left))
+    )
+    (property "Footprint" "Capacitor_SMD:C_0402_1005Metric" (at 102.5652 80.01 0)
+      (effects (font (size 1.27 1.27)) hide)
+    )
+    (property "Datasheet" "~" (at 101.6 76.2 0)
+      (effects (font (size 1.27 1.27)) hide)
+    )
+    (property "Coefficient" "X7R" (at 105.41 78.74 0)
+      (effects (font (size 1.27 1.27)) (justify left))
+    )
+    (property "Voltage" "50V" (at 101.6 76.2 0)
+      (effects (font (size 1.27 1.27)) hide)
+    )
+    (property "Part number" "CC0603KRX7R9BB104" (at 101.6 76.2 0)
+      (effects (font (size 1.27 1.27)) hide)
+    )
+    (property "lcsc" "C14663" (at 101.6 76.2 0)
+      (effects (font (size 1.27 1.27)) hide)
+    )
+    (pin "1")
+    (pin "2")
+    (instances
+      (project "main"
+        (path "/71bbf5b6-a913-4747-956a-150714430eae/8c222416-b30d-49c6-bdd9-9c9a8764b515"
+          (reference "C2") (unit 1)
+        )
+        (path "/71bbf5b6-a913-4747-956a-150714430eae/ca3bda99-bde3-405c-8940-a13088a856d3"
+          (reference "C54") (unit 1)
+        )
+      )
+    )
+  )
+  (symbol (lib_id "Device:R") (at 44.45 76.2 0) (unit 1)
+    (in_bom yes) (on_board yes) (dnp no) (fields_autoplaced)
+    (property "Reference" "R56" (at 46.99 74.93 0)
+      (effects (font (size 1.27 1.27)) (justify left))
+    )
+    (property "Value" "0.3" (at 46.99 77.47 0)
+      (effects (font (size 1.27 1.27)) (justify left))
+    )
+    (property "Footprint" "Resistor_SMD:R_2512_6332Metric" (at 42.672 76.2 90)
+      (effects (font (size 1.27 1.27)) hide)
+    )
+    (property "Datasheet" "~" (at 44.45 76.2 0)
+      (effects (font (size 1.27 1.27)) hide)
+    )
+    (property "lcsc" "C176052" (at 44.45 76.2 0)
+      (effects (font (size 1.27 1.27)) hide)
+    )
+    (pin "1")
+    (pin "2")
+    (instances
+      (project "main"
+        (path "/71bbf5b6-a913-4747-956a-150714430eae/ca3bda99-bde3-405c-8940-a13088a856d3"
+          (reference "R56") (unit 1)
+        )
+      )
+    )
+  )
 )

Commit message: DAPLink, FT2232H
Parts:
- removed C2: 0.1u, Capacitor_SMD:C_0402_1005Metric, symbol Device:C
- removed R56: 0.3, Resistor_SMD:R_2512_6332Metric, symbol Device:R
- removed U8: INA219AxDCN, Package_TO_SOT_SMD:SOT-23-8, symbol Sensor_Energy:INA219AxDCN
Other:
- note added: "16-LFCSP (4x4)"
- note added: "ADA4622"
- note added: "ADP151"
- note added: "ADP1708"
- note added: "ADP2504"
- note added: "C207533"
- note added: "C207546"
- note added: "C461000"
- note added: "C493499"
- note added: "C579239"
- note added: "C61006"
- note added: "C638704"
- note added: "C895366"
- note added: "DMN2050LFDB"
- note added: "DMP1009UFDF"
- note added: "EFC6604R"
- note added: "MCP4451"
- note removed: "mAmp-meter"

Commit message: tmp
Parts:
- added Q2, Q3, Q4, Q5: DMN2050L, Package_TO_SOT_SMD:SOT-23, symbol Transistor_FET:DMN2050L
- added R100: 10k, symbol Device:R
- added R102, R104, R71, R94: 1M, symbol Device:R
- added R103: 100k, symbol Device:R
- added R70: 100, symbol Device:R
- added R86: 1k, symbol Device:R
- added U12: MCP4451-xxxx-ST, Package_SO:TSSOP-20_4.4x6.5mm_P0.65mm, symbol Potentiometer_Digital:MCP4451-xxxx-ST
- added U21: ADA4622-4xCP, Package_CSP:Analog_LFCSP-16-1EP_4x4mm_P0.65mm_EP2.35x2.35mm, symbol Amplifier_Operational:ADA4622-4xCP
Connections:
- new net: Q5.3 (D), R103.2
- new net: Q3.3 (D), R86.2
- new net: R100.1, R103.1, R70.1, R86.1
- new net: Q2.3 (D), R70.2
- new net: Q4.3 (D), R100.2
- new net: U21.17 (V+), U21.3 (V+)
- new net GND: Q2.2 (S), Q3.2 (S), Q4.2 (S), Q5.2 (S), R102.2, R104.2, R71.2, R94.2
- new net LOAD_100: Q2.1 (G), R71.1
- new net LOAD_100K: Q5.1 (G), R104.1
- new net LOAD_10K: Q4.1 (G), R102.1
- new net LOAD_1K: Q3.1 (G), R94.1

Commit message: tmp
Parts:
- removed U12: MCP4451-xxxx-ST, Package_SO:TSSOP-20_4.4x6.5mm_P0.65mm, symbol Potentiometer_Digital:MCP4451-xxxx-ST
- added C138, C140, C141, C142, C145, C147, C150: 0.1u, Capacitor_SMD:C_0402_1005Metric, symbol Device:C
- added C139: 10n, Capacitor_SMD:C_0402_1005Metric, symbol Device:C
- added C143, C144, C156, C157, C158: 4.7u, Capacitor_SMD:C_0402_1005Metric, symbol Device:C
- added C146: 1n, Capacitor_SMD:C_0402_1005Metric, symbol Device:C
- added C148, C149, C151, C152, C153, C154: 470p, Capacitor_SMD:C_0402_1005Metric, symbol Device:C
- added C155, C161: 1u, Capacitor_SMD:C_0402_1005Metric, symbol Device:C
- added C159, C160, C164: 10u, Capacitor_SMD:C_0402_1005Metric, symbol Device:C
- added C162, C163: 2.2u, Capacitor_SMD:C_0402_1005Metric, symbol Device:C
- added D36, D38: PMEG2005AELD, symbol Device:D_Schottky
- added L17, L18: 4.7u, symbol Device:L
- added Q18, Q24, Q25, Q26, Q29, Q30, Q31, Q32, Q33, Q38, Q39, Q40, Q41: NMOS, symbol Simulation_SPICE:NMOS
- added Q34, Q35, Q36, Q37: PMOS, symbol Simulation_SPICE:PMOS
- added R109, R131, R135, R169: 100k, Resistor_SMD:R_0402_1005Metric, symbol Device:R
- added R110, R130, R134: 1M, Resistor_SMD:R_0402_1005Metric, symbol Device:R
- added R136: 110, Resistor_SMD:R_0402_1005Metric, symbol Device:R
- added R137, R139, R140, R143, R145, R146, R147, R148: 47, Resistor_SMD:R_0402_1005Metric, symbol Device:R
- added R138, R168, R178: 1k, Resistor_SMD:R_0402_1005Metric, symbol Device:R
- added R141: 11, Resistor_SMD:R_0402_1005Metric, symbol Device:R
- added R142: 1, Resistor_SMD:R_0402_1005Metric, symbol Device:R
- added R144: 0, Resistor_SMD:R_0402_1005Metric, symbol Device:R
- added R149, R150, R151, R152, R153, R157: 4.7k, Resistor_SMD:R_0402_1005Metric, symbol Device:R
- added R154, R155, R160, R161, R196: 20k, Resistor_SMD:R_0402_1005Metric, symbol Device:R
- added R156: 2.1k, Resistor_SMD:R_0402_1005Metric, symbol Device:R
- added R158, R159, R162, R163, R176: 10k, Resistor_SMD:R_0402_1005Metric, symbol Device:R
- added R164, R165, R172, R173, R183, R184, R187, R188: 8k2, Resistor_SMD:R_0402_1005Metric, symbol Device:R
- added R166, R170, R181, R185: 3k, Resistor_SMD:R_0402_1005Metric, symbol Device:R
- added R167, R171, R182, R186: 6.8k, Resistor_SMD:R_0402_1005Metric, symbol Device:R
- added R174: 560, Resistor_SMD:R_0402_1005Metric, symbol Device:R
- added R175: 330k, Resistor_SMD:R_0402_1005Metric, symbol Device:R
- added R177: 68k, Resistor_SMD:R_0402_1005Metric, symbol Device:R
- added R179, R189, R191, R193: 120k, Resistor_SMD:R_0402_1005Metric, symbol Device:R
- added R180, R190, R192, R194: 30k, Resistor_SMD:R_0402_1005Metric, symbol Device:R
- added R195: 180k, Resistor_SMD:R_0402_1005Metric, symbol Device:R
- added R197: 160k, Resistor_SMD:R_0402_1005Metric, symbol Device:R
- added R198: 560k, Resistor_SMD:R_0402_1005Metric, symbol Device:R
- added R199, R200: 56k, Resistor_SMD:R_0402_1005Metric, symbol Device:R
- added TH2: 10k, symbol Device:Thermistor_NTC
- added U21: ADA4622-4xCP, Package_CSP:Analog_LFCSP-16-1EP_4x4mm_P0.65mm_EP2.35x2.35mm, symbol Amplifier_Operational:ADA4622-4xCP
- added U21: MCP4451-104E/ML, Package_DFN_QFN:QFN-20-1EP_4x4mm_P0.5mm_EP2.7x2.7mm, symbol chrns_ic_analog:MCP443X/5X
- added U26: ADP7118ACPZN, Package_CSP:LFCSP-6-1EP_2x2mm_P0.65mm_EP1x1.6mm, symbol Regulator_Linear:ADP7118ACPZN
- added U27: ADP151, Package_CSP:LFCSP-6-1EP_2x2mm_P0.65mm_EP1x1.6mm, symbol Regulator_Linear:ADP7118ACPZN
- added U29: ADP5072ACBZ-R7, Package_CSP:WLCSP-20_1.934x2.434mm_Layout4x5_P0.4mm, symbol chrns_ic_power:ADP5072
- R100, R102, R103, R104, R70, R71, R86, R94: footprint (none) -> Resistor_SMD:R_0402_1005Metric
Connections:
- net GND: now also U21.10 (V-), C143.2, C144.2, C145.2, C146.2, C149.2, C150.2, C152.2, C156.2, C157.2, C158.2, C159.2, C160.1, C161.1, C162.2, C163.2, C164.2, D38.2 (A), L18.1, Q25.3 (S), Q26.3 (S), Q31.3 (S), Q38.3 (S), Q39.3 (S), Q40.3 (S), Q41.3 (S), R163.1, R177.2, R180.2, R190.2, R192.2, R194.2, R196.2, R198.2, TH2.2, U21.1 (P3B), U21.11 (P0B), U21.14 (A1), U21.16 (P2B), U21.2 (HVC/A0), U21.21 (PAD), U21.5 (VSS), U21.6 (P1B), U26.3 (GND), U26.5 (SS), U26.7 (GND), U27.3 (GND), U27.5 (SS), U27.7 (GND), U29.A4 (PGND), U29.B4 (PGND), U29.D1 (AGND), U29.D2 (SLEW)
- net at U21.11 (+): now also R159.2, R161.1
- net at U21.12 (-): now also R158.2, R160.2
- net SE_OUT: now reaches U21.14
- net SE_OUT: now also R161.2, R162.2, R168.1
- net VREF_IA: now reaches U21.1 (-)
- net VREF_IA: now also U21.15, R160.1
- net IA_OFFSET: now reaches U21.2 (+)
- net IA_OFFSET: now also U21.17 (P2W)
- net VDUT-: now reaches R100.1, R103.1, R70.1, R86.1
- net VDUT-: now also C138.2, C139.2, C140.2, C141.2, C142.2, C144.1, Q18.3 (S), R136.2, R138.2, R141.2, R142.2, R144.2
- net at U21.7: now also R154.2, R158.1
- net at U21.8 (-): now also R154.1, R156.1
- net at U21.9 (+): now also R153.2
- net at U21.4 (+): now also R157.2
- net at U21.5 (-): now also R155.1, R156.2
- net at U21.6: now also R155.2, R159.1
- net 7V0: now reaches U21.17 (V+), U21.3 (V+)
- net 7V0: now also C145.1
- new net: D38.1 (K), L18.2, U29.A2 (SW2)
- new net: Q32.1 (D), Q33.1 (D)
- new net: Q31.1 (D), Q32.2 (G), Q33.2 (G), R135.2
- new net: R164.2, U21.1 (-)
- new net: C148.1, R165.1, R166.1, R167.2, U21.2 (+)
- new net: Q26.1 (D), Q29.2 (G), Q30.2 (G), R131.2
- new net: Q18.1 (D), Q24.1 (D)
- new net: Q18.2 (G), Q24.2 (G), Q25.1 (D), R109.2
- new net: R175.2, R177.1, R178.1, U26.2 (SENSE/ADJ)
- new net: Q35.2 (G), R139.1
- new net: R172.2, U21.4 (+)
- new net: C151.1, R170.1, R171.2, R173.1, U21.5 (-)
- new net: Q29.1 (D), Q30.1 (D)
- new net: C142.1, Q37.3 (S), R144.1
- new net: C141.1, Q35.3 (S), R141.1
- new net: C138.1, Q34.3 (S), R136.1
- new net: Q41.2 (G), R148.2
- new net: R195.2, R196.1, U29.D4 (FB1)
- new net: C149.1, C153.1, R164.1, R168.2, R172.1, R181.1, R182.2, R183.1, R184.1, R187.1, U21.8 (-)
- new net: R183.2, U21.9 (+)
- new net: C140.1, Q36.3 (S), R142.1
- new net: Q34.2 (G), R137.1
- new net: C161.2, R197.1, U29.E3 (VREF)
- new net: C155.2, R178.2
- new net: D36.2 (A), L17.2, U29.A3 (SW1), U29.B3 (SW1)
- new net: R187.2, U21.11 (+)
- new net: C154.1, R185.1, R186.2, R188.1, U21.12 (-)
- new net: Q37.2 (G), R143.1
- new net: Q39.2 (G), R146.2
- new net: R169.2, U21.13 (~{RESET})
- new net: Q36.2 (G), R140.1
- new net: C162.1, R199.2
- new net: R199.1, U29.E1 (COMP2)
- new net: Q40.2 (G), R147.2
- new net: R197.2, R198.1, U29.E2 (FB2)
- new net: R200.1, U29.E4 (COMP1)
- new net: R174.2, U21.18 (P2A)
- new net: C163.1, R200.2
- new net: Q38.2 (G), R145.2
- new net 3V3: C150.1, C157.1, R110.1, R130.1, R134.1, R149.1, R150.1, R151.1, R152.1, R169.1, R174.1, R176.1, U21.15 (VDD), U21.19 (P3A), U21.8 (P1A), U21.9 (P0A), U27.1 (VOUT)
- new net 8V: R109.1, R131.1, R135.1
- new net ANA_EN: U29.C1 (EN2)
- new net AUTO_SW1: C139.1, C143.1, Q30.3 (S), Q33.3 (S), Q34.1 (D), R137.2, R138.1, R145.1, R153.1, R157.1, R165.2, R170.2, R193.1, U21.15
- new net AUTO_SW2: Q35.1 (D), R139.2, R146.1, R167.1, R173.2, R181.2, U21.6
- new net AUTO_SW3: Q36.1 (D), R140.2, R147.1, R171.1, R184.2, R185.2, U21.7
- new net AUTO_SW4: Q37.1 (D), R143.2, R148.1, R182.1, R188.2, U21.14
- new net BB_ADJ: U21.10 (P0W)
- new net DAC: U21.20 (P3W)
- new net EXT_PWR_I: Q29.3 (S)
- new net EXT_PWR_O: Q24.3 (S)
- new net IA_SE_OUT: C146.1, R162.1, R163.2
- new net LDO_ADJ: U21.7 (P1W)
- new net N2V0: C147.2, C148.2, C151.2, C153.2, C154.2, C160.2, R166.2, U21.10 (V-)
- new net NRF_SCL: U21.3 (SCL)
- new net NRF_SDA: U21.4 (SDA)
- new net OUT_EN: Q25.2 (G), R110.2
- new net P0.30/AIN6_NTC: R176.2, TH2.1
- new net P7V0: C147.1, C155.1, C156.1, R175.1, R186.1, U21.17 (V+), U21.3 (V+), U26.1 (VOUT)
- new net P8V0: C152.1, C159.1, D36.1 (K), R195.1, U26.4 (EN), U26.6 (VIN)
- new net SW1_ONOFF: Q38.1 (D), R149.2
- new net SW2_ONOFF: Q39.1 (D), R150.2
- new net SW3_ONOFF: Q40.1 (D), R151.2
- new net SW4_ONOFF: Q41.1 (D), R152.2
- new net VBB: R189.1
- new net VBB_SNS: R189.2, R190.1
- new net VDUT_SNS: R193.2, R194.1
- new net VEXT_EN: Q26.2 (G), R130.2
- new net VIN: C158.1, C164.1, L17.1, R191.1, U27.4 (EN), U27.6 (VIN), U29.A1 (PVIN), U29.B1 (AVIN), U29.B2 (PVIN), U29.C2 (SYNC), U29.C3 (SEQ), U29.C4 (EN1)
- new net VLDO: Q32.3 (S), R179.1
- new net VLDO_EN: Q31.2 (G), R134.2
- new net VLDO_SNS: R179.2, R180.1
- new net VLIN_SNS: R191.2, R192.1
- no-connect marks 0 -> 2
Other:
- note added: "ADP5072ACBZ-R7"
- note added: "C637740"
- note added: "DAC"
- note added: "Input supply: 2.2V - 5.5V Output Current: 200mA PSRR: 70dB @ 10kHz Vdrop: 135mV@200mA Fixed 3.3"
- note added: "Input supply: 2.7V - 20V Output Current: 200mA PSRR: 88dB @ 10kHz Vdrop: 200mV Vout = 1.2 * (1 + 330k/68k) = 7.02V"
- note added: "Input supply: 2.85V - 5.5V"
- note added: "MCP4451-104E/ML"
- note added: "Vneg = Vfb2 - (Rft2/Rfb2)*(Vref-Vfb2) Vneg = 0.8V - (560k/160k)*(1.6V - 0.8V) = -2V"
- note added: "Vpos = Vfb1 * (1 + Rft1/Rfb1)) Vpos = 0.8V * (1 + 180k/20k) = 8V"
- moved on the sheet: Q2, Q3, Q4, Q5, R100, R102, R103, R104, R70, R71, R86, R94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
